File: hardware/Buck_Converter.kicad_sch (KiCad schematic)
At the start: 40 parts, among them U7 EA3059

Commit message: feat(Hw):Update_Schematic
Parts:
- C11, C16, C7, C9: LCSC# C327000 -> C107001
Changed lines of the file:
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@@
 			)
 		)
-		(property "LCSC#" "C327000"
+		(property "LCSC#" "C107001"
 			(at 177.8 71.12 0)
 			(effects
@@
 			)
 		)
-		(property "LCSC#" "C327000"
+		(property "LCSC#" "C107001"
 			(at 175.26 119.38 0)
 			(effects
@@
 			)
 		)
-		(property "LCSC#" "C327000"
+		(property "LCSC#" "C107001"
 			(at 233.68 120.65 0)
 			(effects
@@
 			)
 		)
-		(property "LCSC#" "C327000"
+		(property "LCSC#" "C107001"
 			(at 236.22 71.12 0)
 			(effects
