File: hardware/Wifi_Module.kicad_sch (KiCad schematic)
At the start: 36 parts, among them J5 Conn_Coaxial, U2 AP6256, Y3 37.4 Mhz, Y4 OK2EL89CJI-111YLC-32.768K

Commit message: feat(Hw):Update_Schematic
Parts:
- C22, C31: #LCSC C415703 -> (none); LCSC# (none) -> C415703; Mnfr# GRM155R60J226ME11D -> (none); manf# (none) -> GRM155R60J226ME11D
- C32, C33: #LCSC C524558 -> (none); LCSC# (none) -> C524558
- C37: #LCSC C162274 -> (none); LCSC# (none) -> C162274
- C44: #LCSC C326803 -> (none); LCSC# (none) -> C326803
- C45: #LCSC C96446 -> (none); LCSC# (none) -> C96446
- C50, C53: #LCSC C77020 -> (none); LCSC# (none) -> C77020
- FB3: #LCSC C79382 -> (none); LCSC# (none) -> C79382
- J5: Mnfr# CONMHF1-SMD-G-T -> (none); manf# (none) -> CONMHF1-SMD-G-T
- L1: #LCSC C279952 -> (none); LCSC# (none) -> C279952; Mnfr# WPN252010U1R0MT -> (none); manf# (none) -> WPN252010U1R0MT
- R44, R59: #LCSC C400631 -> (none); LCSC# (none) -> C400631
- R45, R46, R47, R48, R49, R52, R53, R54, R56, R57, R58, R61, R62, R63, R64: #LCSC C2759535 -> (none); LCSC# (none) -> C2759535
- R50: #LCSC C844674 -> (none); LCSC# (none) -> C844674
- R55, R60: #LCSC C242161 -> (none); LCSC# (none) -> C242161
- U2: #LCSC C5248079 -> (none); LCSC# (none) -> C5248079
- U4: Mnfr# NDC7002N -> (none); manf# (none) -> NDC7002N
- Y3: #LCSC C655049 -> (none); LCSC# (none) -> C655049
- Y4: #LCSC C5280579 -> (none); LCSC# (none) -> C5280579; Mnfr# OK2EL89CJI-111YLC-32.768K -> (none); manf# (none) -> OK2EL89CJI-111YLC-32.768K

Commit message: feat(Hw):Update_Schematic
Parts:
- Y3: footprint pondo_2:SMD1612-4P -> Footprints:SMD1612-4P
Changed lines of the file:
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@@
 			)
 		)
-		(property "Datasheet" "C400631"
+		(property "Datasheet" ""
 			(at 111.76 152.4 0)
 			(effects
@@
 			)
 		)
-		(property "Datasheet" "C400631"
+		(property "Datasheet" ""
 			(at 118.11 152.4 0)
 			(effects
@@
 			)
 		)
-		(property "Footprint" "pondo_2:SMD1612-4P"
+		(property "Footprint" "Footprints:SMD1612-4P"
 			(at 191.77 36.83 0)
 			(effects
