File: hardware/Badge_Bugcon_2025.kicad_pcb (KiCad board)
At the start: 2 copper layers, 109 parts, among them J1 Conn_01x10_Pin, J2 Conn_01x04_Pin, J4 Conn_01x03, P4 USB_C_Plug_USB2.0, SW2 SW_Push, SW3 SW_Push, U6 W25N02KVZEIR, U7 EA3059, Y1 Crystal, Y2 24MHz

Commit message: feat(Hw):Update_Schematic
Parts:
- moved C51 121.6 mm to (210.9, 95.4)
- moved C11 116.9 mm to (20.9, 93.8)
- moved C12 116.9 mm to (20.9, 95.7)
- moved C52 114.8 mm to (210.9, 94.2)
- moved R6 110.9 mm to (32.1, 89.9)
- moved R21 110.9 mm to (35.4, 91.9)
- moved L6 107.5 mm to (28.3, 94.0)
- moved R35 96.2 mm to (210.9, 96.6)
- moved L4 88.1 mm to (44.0, 59.6)
- moved L5 88.1 mm to (44.0, 63.3)
- moved L7 88.1 mm to (44.0, 70.8)
- moved U7 88.1 mm to (49.7, 81.6)
- moved C13 88.1 mm to (51.4, 67.7)
- moved C14 88.1 mm to (51.4, 69.6)
- moved C15 88.1 mm to (51.4, 71.6)
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
Commit message: feat(Hw):Update_Schematic
Parts:
- added BT1: Battery_Cell, Battery:BatteryHolder_Keystone_2466_1xAAA, F.Cu at (167.9, -50.5)
- added BT2: Battery_Cell, Battery:BatteryHolder_Keystone_2466_1xAAA, F.Cu at (167.9, -36.5)
- added BT3: Battery_Cell, Battery:BatteryHolder_Keystone_2466_1xAAA, F.Cu at (167.8, -22.5)
- added C18: 10uF, Capacitor_SMD:C_0402_1005Metric, F.Cu at (144.9, 28.7)
- added C2: 100nF, Capacitor_SMD:C_0603_1608Metric, F.Cu at (144.9, 41.0)
- added C21: 100nF, Capacitor_SMD:C_0603_1608Metric, F.Cu at (144.9, 43.5)
- added C22: 22uf, Capacitor_SMD:C_0402_1005Metric_Pad0.74x0.62mm_HandSolder, F.Cu at (123.5, 40.8)
- added C31: 22uf, Capacitor_SMD:C_0402_1005Metric_Pad0.74x0.62mm_HandSolder, F.Cu at (123.5, 42.7)
- added C32: 14pf, Capacitor_SMD:C_0402_1005Metric_Pad0.74x0.62mm_HandSolder, F.Cu at (123.5, 44.7)
- added C33: 14pf, Capacitor_SMD:C_0402_1005Metric_Pad0.74x0.62mm_HandSolder, F.Cu at (123.5, 46.7)
- added C37: 4.7uf, Capacitor_SMD:C_0603_1608Metric_Pad1.08x0.95mm_HandSolder, F.Cu at (138.5, 58.3)
- added C43: 100nF, Capacitor_SMD:C_0603_1608Metric, F.Cu at (144.9, 46.1)
- added C44: 15pf, Capacitor_SMD:C_0402_1005Metric_Pad0.74x0.62mm_HandSolder, F.Cu at (123.5, 48.6)
- added C45: 10uF, Capacitor_SMD:C_0603_1608Metric, F.Cu at (138.4, 51.0)
- added C46: 100nF, Capacitor_SMD:C_0603_1608Metric, F.Cu at (144.9, 48.6)
- added C47: 100nF, Capacitor_SMD:C_0603_1608Metric, F.Cu at (144.9, 51.1)
- added C50: 100nF, Capacitor_SMD:C_0402_1005Metric_Pad0.74x0.62mm_HandSolder, F.Cu at (123.5, 50.6)
- added C53: 100nF, Capacitor_SMD:C_0402_1005Metric_Pad0.74x0.62mm_HandSolder, F.Cu at (123.5, 52.6)
- added C54: 100nF, Capacitor_SMD:C_0402_1005Metric, F.Cu at (144.9, 30.7)
- added D10: WS2812E-1313, Footprints:WS2812E-1313, F.Cu at (148.8, 50.3)
- added D11: WS2812E-1313, Footprints:WS2812E-1313, F.Cu at (148.8, 53.3)
- added D12: MBR120, Diode_SMD:D_SOD-123F, F.Cu at (135.8, 32.8)
- added D13: 1N5817, Diode_SMD:D_SOD-123F, F.Cu at (135.8, 36.1)
- added D2: 1N5817, Diode_SMD:D_SOD-123F, F.Cu at (135.8, 29.4)
- added D7: WS2812E-1313, Footprints:WS2812E-1313, F.Cu at (148.8, 41.2)
- added D8: WS2812E-1313, Footprints:WS2812E-1313, F.Cu at (148.8, 44.2)
- added D9: WS2812E-1313, Footprints:WS2812E-1313, F.Cu at (148.8, 47.2)
- added F1: 750mA, Fuse:Fuse_0603_1608Metric, F.Cu at (80.2, 27.5)
- added F2: 750mA, Fuse:Fuse_0603_1608Metric, F.Cu at (80.2, 30.0)
- added FB3: BLM21PG121SN1D, Inductor_SMD:L_0805_2012Metric, F.Cu at (138.6, 55.7)
- added J1: Flash, Connector_PinHeader_2.54mm:PinHeader_1x08_P2.54mm_Vertical, F.Cu at (155.0, 42.1)
- added J5: Conn_Coaxial, Connector_Coaxial:U.FL_Molex_MCRF_73412-0110_Vertical, F.Cu at (128.1, 52.9)
- added L1: 1uH, Inductor_SMD:L_1008_2520Metric, F.Cu at (127.6, 57.7)
- added P4: USB_C_Plug_USB2.0, Footprints:C393939, F.Cu at (127.5, 29.9)
- added Q1: DMG3415U-7, Package_TO_SOT_SMD:SOT-23, F.Cu at (141.0, 30.1)
- added R11: 100K, Resistor_SMD:R_0603_1608Metric, F.Cu at (80.2, 32.5)
- added R13: 10K, Resistor_SMD:R_0402_1005Metric, F.Cu at (140.0, 33.4)
- added R14: 5k1, Resistor_SMD:R_0603_1608Metric, F.Cu at (80.2, 35.0)
- added R15: 5k1, Resistor_SMD:R_0603_1608Metric, F.Cu at (80.2, 37.5)
- added R19: 18k, Resistor_SMD:R_0402_1005Metric, F.Cu at (140.0, 35.3)
- added R4: 470R, Resistor_SMD:R_0603_1608Metric, F.Cu at (144.9, 53.6)
- added R44: 4.7K, Resistor_SMD:R_0402_1005Metric_Pad0.72x0.64mm_HandSolder, F.Cu at (126.8, 40.8)
- added R45: 10K, Resistor_SMD:R_0402_1005Metric_Pad0.72x0.64mm_HandSolder, F.Cu at (126.8, 42.8)
- added R46: 10K, Resistor_SMD:R_0402_1005Metric_Pad0.72x0.64mm_HandSolder, F.Cu at (126.8, 44.8)
- added R47: 10K, Resistor_SMD:R_0402_1005Metric_Pad0.72x0.64mm_HandSolder, F.Cu at (126.8, 46.8)
- added R48: 10K, Resistor_SMD:R_0402_1005Metric_Pad0.72x0.64mm_HandSolder, F.Cu at (126.8, 48.7)
- added R49: 10K, Resistor_SMD:R_0402_1005Metric_Pad0.72x0.64mm_HandSolder, F.Cu at (130.0, 40.8)
- added R50: 100K, Resistor_SMD:R_0402_1005Metric_Pad0.72x0.64mm_HandSolder, F.Cu at (130.0, 42.8)
- added R52: 10K, Resistor_SMD:R_0402_1005Metric_Pad0.72x0.64mm_HandSolder, F.Cu at (130.0, 44.8)
- added R53: 10K, Resistor_SMD:R_0402_1005Metric_Pad0.72x0.64mm_HandSolder, F.Cu at (130.0, 46.8)
- added R54: 10K, Resistor_SMD:R_0402_1005Metric_Pad0.72x0.64mm_HandSolder, F.Cu at (130.0, 48.7)
- added R55: 1K, Resistor_SMD:R_0402_1005Metric_Pad0.72x0.64mm_HandSolder, F.Cu at (133.3, 40.8)
- added R56: 10K, Resistor_SMD:R_0402_1005Metric_Pad0.72x0.64mm_HandSolder, F.Cu at (133.3, 42.8)
- added R57: 10K, Resistor_SMD:R_0402_1005Metric_Pad0.72x0.64mm_HandSolder, F.Cu at (133.3, 44.8)
- added R58: 10K, Resistor_SMD:R_0402_1005Metric_Pad0.72x0.64mm_HandSolder, F.Cu at (133.3, 46.8)
- added R59: 4.7K, Resistor_SMD:R_0402_1005Metric_Pad0.72x0.64mm_HandSolder, F.Cu at (133.3, 48.7)
- added R60: 1K, Resistor_SMD:R_0402_1005Metric_Pad0.72x0.64mm_HandSolder, F.Cu at (136.6, 40.8)
- added R61: 10K, Resistor_SMD:R_0402_1005Metric_Pad0.72x0.64mm_HandSolder, F.Cu at (136.6, 42.8)
- added R62: 10K, Resistor_SMD:R_0402_1005Metric_Pad0.72x0.64mm_HandSolder, F.Cu at (136.6, 44.8)
- added R63: 10K, Resistor_SMD:R_0402_1005Metric_Pad0.72x0.64mm_HandSolder, F.Cu at (136.6, 46.8)
- added R64: 10K, Resistor_SMD:R_0402_1005Metric_Pad0.72x0.64mm_HandSolder, F.Cu at (136.6, 48.7)
- added U4: ~, Package_TO_SOT_SMD:SuperSOT-6, F.Cu at (133.7, 56.7)
- added Y3: 37.4 Mhz, Footprints:SMD1612-4P, F.Cu at (123.4, 54.9)
- added Y4: OK2EL89CJI-111YLC-32.768K, Crystal:Crystal_SMD_3225-4Pin_3.2x2.5mm, F.Cu at (133.8, 52.0)
- C1: footprint Capacitor_SMD:C_0603_1608Metric_Pad1.08x0.95mm_HandSolder -> Capacitor_SMD:C_0603_1608Metric
- C10, C11, C12, C13, C14, C15, C16, C17, C20, C23, C25, C26, C27, C29, C3, C30, C35, C36, C39, C4, C40, C41, C42, C49, C5, C52, C6, C63, C65, C7, C8, C9: footprint Capacitor_SMD:C_0402_1005Metric_Pad0.74x0.62mm_HandSolder -> Capacitor_SMD:C_0402_1005Metric
- R1, R10, R12, R18, R2, R20, R21, R22, R23, R24, R26, R28, R29, R30, R33, R35, R36, R38, R5, R6, R7, R8, R9: footprint Resistor_SMD:R_0402_1005Metric_Pad0.72x0.64mm_HandSolder -> Resistor_SMD:R_0402_1005Metric
Connections:
- net /MCU/CSI_SCK renamed /MCU/GPIO3_C7_D
- net /MCU/CSI_SDA renamed /MCU/GPIO3_D0_D
- net /MCU/DIN renamed /MCU/GPIO4_A1_U
- net /MCU/INT renamed /MCU/GPIO0_A4_D
- net /MCU/IR_SCL renamed /MCU/GPIO1_A0_D
- net /MCU/IR_SDA renamed /MCU/GPIO1_A1_D
- net /MCU/Lineout renamed /MCU/CODEC_LINEOUT
- net /MCU/MCSI_CKN renamed /MCU/GPIO3_C0_D
- net /MCU/MCSI_CKP renamed /MCU/GPIO3_C1_D
- net /MCU/MCSI_D0N renamed /MCU/GPIO3_C2_D
- net /MCU/MCSI_D0P renamed /MCU/GPIO3_C3_D
- net /MCU/MCSI_D1N renamed /MCU/GPIO3_B6_D
- net /MCU/MCSI_D1P renamed /MCU/GPIO3_B7_D
- net /MCU/MCSI_RST renamed /MCU/GPIO3_C5_D
- net /MCU/MIC+ renamed /MCU/CODEC_MIC0P
- net /MCU/MIC- renamed /MCU/CODEC_MIC0N
- net /MCU/MICBIAS renamed /MCU/CODEC_MICBIAS
- net /MCU/Sound_En renamed /MCU/GPIO1_D3_D
- U8 pad 100: unconnected-(U8D-ETH_PHY_TXP-Pad100) -> /MCU/ETH_PHY_TXP
- U8 pad 102: unconnected-(U8D-ETH_EXTR-Pad102) -> /MCU/ETH_EXTR
- U8 pad 104: unconnected-(U8D-UART0_TX_M1/I2C1_SDA_M1/VO_LCDC_D17/PWM6_M1_/GPIO2_B1_D_1-Pad104) -> /MCU/GPIO2_B1_D_1
- U8 pad 105: unconnected-(U8D-UART0_TX_M1/I2C1_SDA_M1/VO_LCDC_D17/PWM6_M1_/GPIO2_B1_D_2-Pad105) -> /MCU/GPIO2_B1_D_2
- U8 pad 106: unconnected-(U8D-UART0_CTS_M1/I2S0_SDO1_SDI3/VO_LCDC_D15/PWM_4_M1/I2C3_SDA_M0/PRELIGHT_TRIG_OUT/GPIO2_A7_D-Pad106) -> /MCU/GPIO2_A7_D
- U8 pad 107: unconnected-(U8D-UART0_RTS_M1/I2S0_SDO2_SDI2/VO_LCDC_D14/PWM_2_M1/I2C3_SCL_M0/FLASH_TRIG_OUT/GPIO2_A6_D-Pad107) -> /MCU/GPIO2_A6_D
- U8 pad 109: unconnected-(U8D-SDMMC1_D1_M0/I2S0_SCLK/VO_LCDC_D8/UART1_CTS__M1/I2C4_SDA_M0/GPIO2_A0_D_1-Pad109) -> /MCU/GPIO2_A0_D_1
- U8 pad 110: unconnected-(U8D-SDMMC1_D1_M0/I2S0_SCLK/VO_LCDC_D8/UART1_CTS__M1/I2C4_SDA_M0/GPIO2_A0_D_2-Pad110) -> /MCU/GPIO2_A0_D_2
- U8 pad 111: unconnected-(U8D-SDMMC1_CLK_M0/I2S0_MCLK/VO_LCDC_D10/GPIO2_A_2_D-Pad111) -> /MCU/GPIO2_A_2_D
- U8 pad 112: /MCU/GPIO -> /MCU/GPIO2_A3_D
- U8 pad 113: unconnected-(U8D-SDMMC1_D3_M0/I2S0_SDO0/VO_LCDC_D12/UART1_TX__M1/GPIO2_A4_D-Pad113) -> /MCU/GPIO2_A4_D
- U8 pad 114: unconnected-(U8D-SDMMC1_D2_M0/I2S0_SDI0/VO_LCDC_D13/UART1_RX__M1/GPIO2_A5_D-Pad114) -> /MCU/GPIO2_A5_D
- U8 pad 119: unconnected-(U8D-VI_CIF_D2_M0/MIPI_CSI_RX_CK1N/LVDS_RX_CK1N/GP_IO3_B2_D-Pad119) -> /MCU/GPIO3_B2_D
- U8 pad 120: unconnected-(U8D-VI_CIF_D3_M0/MIPI_CSI_RX_CK1P/LVDS_RX_CK1P/GPI_O3_B3_D-Pad120) -> /MCU/GPIO3_B3_D
- U8 pad 121: unconnected-(U8D-VI_CIF_D4_M0/MIPI_CSI_RX_D2N/LVDS_RX_D2N/GPIO_3_B4_D-Pad121) -> /MCU/GPIO3_B4_D
- U8 pad 122: unconnected-(U8D-VI_CIF_D5_M0/MIPI_CSI_RX_D2P/LVDS_RX_D2P/GPIO3__B5_D-Pad122) -> /MCU/GPIO3_B5_D
- U8 pad 2: Net-(U8A-VI_CIF_CLKO_M0/MIPI_CLK0_OUT/GPIO3_C4_D) -> /MCU/GPIO3_C4_D
- U8 pad 22: unconnected-(U8A-SARADC_IN1/PWM1_M1/GPI4_C1_Z-Pad22) -> /MCU/GPIO4_C1_Z
- U8 pad 35: unconnected-(U8B-CODEC_MIC1N-Pad35) -> /MCU/CODEC_MIC1N
- U8 pad 36: unconnected-(U8B-CODEC_MIC1P-Pad36) -> /MCU/CODEC_MIC1P
- U8 pad 38: unconnected-(U8B-EMMC_D5/SPI1_CLK_M0/UART1_RX_M2/I2C2_SCL_M1/GPIO4__A7_U-Pad38) -> /MCU/GPIO4_A7_U
- U8 pad 40: unconnected-(U8B-EMMC_D4/SPI1_CS0_M0/UART1_TX_M2/I2C2_SDA_M1/GPIO4__A5_U-Pad40) -> /MCU/GPIO4_A5_U
- U8 pad 46: unconnected-(U8B-EMMC_D7/SPI1_MISO_M0/UART0_RX_M2/I2C0_SDA_M1/GPIO_4_A0_U-Pad46) -> /MCU/GPIO4_A0_U
- U8 pad 58: /Buck_Converter/POGO_TX -> /MCU/GPIO0_A0_Z
- U8 pad 59: /Buck_Converter/POGO_RX -> /MCU/GPIO0_A1_D
- U8 pad 6: unconnected-(U8A-VI_CIF_D13/UART5_RTS_M2/I2C3_SCL_M2/GPIO3_D1_D-Pad6) -> /MCU/GPIO3_D1_D
- U8 pad 62: unconnected-(U8B-PMIC_PWR_CTRL_M1/GPIO0_A3_U-Pad62) -> /MCU/GPIO0_A3_U
- U8 pad 74: /MCU/WL_REG_ON -> /Wifi_Module/WL_EN
- U8 pad 77: unconnected-(U8C-UART4_RX_M0/PWM3_IR_M1/GPIO1_B0_D-Pad77) -> /MCU/GPIO1_B0_D
- U8 pad 8: unconnected-(U8A-VI_CIF_D14/UART5_CTS_M2/I2C3_SDA_M2/GPIO3_D2_D-Pad8) -> /MCU/GPIO3_D2_D
- U8 pad 83: unconnected-(U8C-VO_LCDC_D1/VI_CIF_D8_M1/PWM10_M1/UART4_RTS__M1/GPIO1_C6_D-Pad83) -> /MCU/GPIO1_C6_D
- U8 pad 84: unconnected-(U8C-VO_LCDC_D0/VI_CIF_D9_M1/PWM11_IR_M1/UART4_CT_S_M1/GPIO1_C7_D-Pad84) -> /MCU/GPIO1_C7_D
- U8 pad 86: unconnected-(U8C-VO_LCDC_VSYNC/VI_CIF_VSYNC_M1/I2C3_SDA_M1/UA_RT5_RX_M1/SPI0_CS1_M0/PWM0_M1/AUD_DSM_P/GPI_O1_D2_D-Pad86) -> /MCU/GPIO1_D2_D
- U8 pad 87: unconnected-(U8C-VO_LCDC_HSYNC/VI_CIF_HREF_M1/PWM10_M2/UART5__CTS_M1/UART3_RX_M1/GPIO1_D1_D-Pad87) -> /MCU/GPIO1_D1_D
- U8 pad 89: unconnected-(U8C-VO_LCDC_DEN/VI_CIF_CLKI_M1/PWM3_IR_M2/UART5__RTS_M1/UART3_TX_M1/GPIO1_D0_D-Pad89) -> /MCU/GPIO1_D0_D
- U8 pad 9: unconnected-(U8A-VI_CIF_D15/PWM1_M2/GPIO3_D3_D-Pad9) -> /MCU/GPIO3_D3_D
- U8 pad 90: unconnected-(U8C-VO_LCDC_D2/VI_CIF_D7_M1/PWM9_M1/UART4_TX_M1/_SDMMC1_D2_M1/GPIO1_C5_D-Pad90) -> /MCU/GPIO1_C5_D
- U8 pad 91: unconnected-(U8C-VO_LCDC_D3/VI_CIF_D6_M1/PWM8_M1/UART4_RX_M1_/SDMMC1_D3_M1/GPIO1_C4_D-Pad91) -> /MCU/GPIO1_C4_D
- U8 pad 92: unconnected-(U8C-VO_LCDC_D4/VI_CIF_D5_M1/PWM6_M2/I2C4_SDA_M1/_SDMMC1_CMD_M1/SPI0_MISO_M0/GPIO1_C3_D-Pad92) -> /MCU/GPIO1_C3_D
- U8 pad 94: unconnected-(U8C-VO_LCDC_D6/VI_CIF_D3_M1/PWM4_M2/SPI0_CLK_M0/_SDMMC1_D0_M1/GPIO1_C1_D-Pad94) -> /MCU/GPIO1_C1_D
- U8 pad 95: unconnected-(U8C-VO_LCDC_D7/VI_CIF_D2_M1/PWM2_M2/SPI0_CS0_M0/_SDMMC1_D1_M1/GPIO1_C0_D-Pad95) -> /MCU/GPIO1_C0_D
- U8 pad 97: unconnected-(U8D-ETH_PHY_RXN-Pad97) -> /MCU/ETH_PHY_RXN
- U8 pad 98: unconnected-(U8D-ETH_PHY_RXP-Pad98) -> /MCU/ETH_PHY_RXP
- U8 pad 99: unconnected-(U8D-ETH_PHY_TXN-Pad99) -> /MCU/ETH_PHY_TXN
