File: hardware/Badge_Bugcon_2025.kicad_sch (KiCad schematic)
At the start: 0 parts

Commit message: feat(Hw):Update_Schematic
Other:
- added sheet Neopixels (Neopixels.kicad_sch)
- added sheet USB (USB.kicad_sch)
- added sheet Wifi_Module (Wifi_Module.kicad_sch)
- sheet Buck_Converter: file untitled.kicad_sch -> Buck_Converter.kicad_sch
- sheet MCU ports: added BT_HOST_WAKE, BT_REG_ON, BT_WAKE, CLK_SDIO, CMD_SDIO, CTS_BT, DAT0_SDIO, DAT1_SDIO, DAT2_SDIO, DAT3_SDIO, DIN_IR, RTS_BT, RX_BT, TX_BT, WL_REG_ON, WT_HOST_WAKE; removed V5V

Commit message: feat(Hw):Update_Schematic
Other:
- sheet MCU ports: added D+, D-; removed none
- sheet USB ports: added D+, D-; removed none
Changed lines of the file:
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@@
+	(wire
+		(pts
+			(xy 77.47 88.9) (xy 125.73 88.9)
+		)
+		(stroke
+			(width 0)
+			(type default)
+		)
+	)
 	(wire
 		(pts
@@
 		(pts
 			(xy 163.83 83.82) (xy 177.8 83.82)
+		)
+		(stroke
+			(width 0)
+			(type default)
+		)
+	)
+	(wire
+		(pts
+			(xy 77.47 86.36) (xy 125.73 86.36)
 		)
 		(stroke
@@
 	(sheet
 		(at 58.42 83.82)
-		(size 18.796 14.986)
+		(size 19.05 14.986)
 		(exclude_from_sim no)
 		(in_bom yes)
@@
 				)
 				(justify left)
+			)
+		)
+		(pin "D+" output
+			(at 77.47 86.36 0)
+			(effects
+				(font
+					(size 1.27 1.27)
+				)
+				(justify right)
+			)
+		)
+		(pin "D-" output
+			(at 77.47 88.9 0)
+			(effects
+				(font
+					(size 1.27 1.27)
+				)
+				(justify right)
 			)
 		)
@@
 			(effects
 				(font
+					(size 1.27 1.27)
+				)
+				(justify left)
+			)
+		)
+		(pin "D+" input
+			(at 125.73 86.36 180)
+			(effects
+				(font
+					(size 1.27 1.27)
+				)
+				(justify left)
+			)
+		)
+		(pin "D-" input
+			(at 125.73 88.9 180)
+			(effects
+				(font

Commit message: feat(Hw):Update_Schematic
Other:
- sheet MCU ports: added USB_DET; removed none
- sheet USB ports: added USB_DET; removed none
Changed lines of the file:
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@@
+	(wire
+		(pts
+			(xy 77.47 91.44) (xy 125.73 91.44)
+		)
+		(stroke
+			(width 0)
+			(type default)
+		)
+	)
 	(wire
 		(pts
@@
 			)
 		)
+		(pin "USB_DET" output
+			(at 77.47 91.44 0)
+			(effects
+				(font
+					(size 1.27 1.27)
+				)
+				(justify right)
+			)
+		)
 		(instances
 			(project "Badge_Bugcon_2025"
@@
 			(effects
 				(font
+					(size 1.27 1.27)
+				)
+				(justify left)
+			)
+		)
+		(pin "USB_DET" input
+			(at 125.73 91.44 180)
+			(effects
+				(font

Commit message: feat(Hw):Update_Schematic
Other:
- added sheet OLED (OLED.kicad_sch)
Changed lines of the file:
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@@
 	(paper "A4")
 	(junction
-		(at 113.03 71.12)
+		(at 118.11 71.12)
 		(diameter 0)
 		(color 0 0 0 0)
 	)
 	(junction
-		(at 109.22 73.66)
+		(at 114.3 73.66)
 		(diameter 0)
 		(color 0 0 0 0)
@@
 	(wire
 		(pts
-			(xy 109.22 102.87) (xy 109.22 73.66)
-		)
-		(stroke
-			(width 0)
-			(type default)
-		)
-	)
-	(wire
-		(pts
-			(xy 82.55 73.66) (xy 109.22 73.66)
-		)
-		(stroke
-			(width 0)
-			(type default)
-		)
-	)
-	(wire
-		(pts
-			(xy 109.22 73.66) (xy 125.73 73.66)
+			(xy 114.3 102.87) (xy 114.3 73.66)
+		)
+		(stroke
+			(width 0)
+			(type default)
+		)
+	)
+	(wire
+		(pts
+			(xy 82.55 73.66) (xy 114.3 73.66)
 		)
 		(stroke
@@
 	(wire
 		(pts
+			(xy 114.3 73.66) (xy 125.73 73.66)
+		)
+		(stroke
+			(width 0)
+			(type default)
+		)
+	)
+	(wire
+		(pts
 			(xy 77.47 91.44) (xy 125.73 91.44)
 		)
@@
 	(wire
 		(pts
-			(xy 102.87 102.87) (xy 109.22 102.87)
-		)
-		(stroke
-			(width 0)
-			(type default)
-		)
-	)
-	(wire
-		(pts
-			(xy 113.03 71.12) (xy 125.73 71.12)
+			(xy 102.87 102.87) (xy 114.3 102.87)
 		)
 		(stroke
@@
 	(wire
 		(pts
+			(xy 118.11 71.12) (xy 125.73 71.12)
+		)
+		(stroke
+			(width 0)
+			(type default)
+		)
+	)
+	(wire
+		(pts
 			(xy 82.55 58.42) (xy 125.73 58.42)
 		)
@@
 	(wire
 		(pts
-			(xy 82.55 71.12) (xy 113.03 71.12)
+			(xy 82.55 71.12) (xy 118.11 71.12)
 		)
 		(stroke
@@
 	(wire
 		(pts
-			(xy 181.61 120.65) (xy 113.03 120.65)
+			(xy 181.61 120.65) (xy 118.11 120.65)
 		)
 		(stroke
@@
 	(wire
 		(pts
-			(xy 113.03 120.65) (xy 113.03 71.12)
+			(xy 118.11 120.65) (xy 118.11 71.12)
 		)
 		(stroke
@@
 		)
 	)
+	(sheet
+		(at 58.674 114.046)
+		(size 19.05 19.05)
+		(exclude_from_sim no)
+		(in_bom yes)
+		(on_board yes)
+		(dnp no)
+		(fields_autoplaced yes)
+		(stroke
+			(width 0.1524)
+			(type solid)
+		)
+		(fill
+			(color 0 0 0 0.0000)
+		)
+		(property "Sheetname" "OLED"
+			(at 58.674 113.3344 0)
+			(effects
+				(font
+					(size 1.27 1.27)
+				)
+				(justify left bottom)
+			)
+		)
+		(property "Sheetfile" "OLED.kicad_sch"
+			(at 58.674 133.6806 0)
+			(effects
+				(font
+					(size 1.27 1.27)
+				)
+				(justify left top)
+			)
+		)
+		(instances
+			(project "Badge_Bugcon_2025"
+				(path "/a95785a0-0aa1-454e-b59f-0ac64970ac71"
+					(page "7")
+				)
+			)
+		)
+	)
