File: hardware/MCU.kicad_sch (KiCad schematic)
At the start: 68 parts, among them J2 Conn_01x04_Pin, J4 Conn_01x03, P4 USB_C_Plug_USB2.0, SW2 SW_Push, SW3 SW_Push, U6 W25N02KVZEIR, Y1 Crystal, Y2 24MHz

Commit message: feat(Hw):Update_Schematic
Parts:
- removed C18: 10uF, Capacitor_SMD:C_0402_1005Metric_Pad0.74x0.62mm_HandSolder, symbol Device:C_Small
- removed C19: 100nF, Capacitor_SMD:C_0402_1005Metric_Pad0.74x0.62mm_HandSolder, symbol Device:C
- removed D2: 1N5817, Diode_SMD:D_SOD-123F, symbol Diode:1N5817
- removed F1: 750mA, Fuse:Fuse_0603_1608Metric, symbol Device:Fuse_Small
- removed J4: Conn_01x03, Connector_PinHeader_2.54mm:PinHeader_1x03_P2.54mm_Vertical, symbol Connector_Generic:Conn_01x03
- removed P4: USB_C_Plug_USB2.0, Footprints:C393939, symbol HunterCat-NFC-rescue:USB_C_Plug_USB2.0-Connector
- removed R14, R15: 5k1, Resistor_SMD:R_0603_1608Metric, symbol Device:R_Small
- removed R31: 10K, Resistor_SMD:R_0402_1005Metric_Pad0.72x0.64mm_HandSolder, symbol Device:R_Small
- removed R32: 18k, Resistor_SMD:R_0402_1005Metric_Pad0.72x0.64mm_HandSolder, symbol Device:R
- added J1: Flash, symbol Connector_Generic:Conn_01x08
- C1: footprint Capacitor_SMD:C_0603_1608Metric_Pad1.08x0.95mm_HandSolder -> Capacitor_SMD:C_0603_1608Metric
- C20, C23, C25, C26, C27, C29, C3, C30, C35, C36, C39, C4, C40, C41, C42, C49, C5, C52, C6, C63, C65: footprint Capacitor_SMD:C_0402_1005Metric_Pad0.74x0.62mm_HandSolder -> Capacitor_SMD:C_0402_1005Metric
- R10, R18, R2, R26, R28, R29, R30, R33, R35, R36, R9: footprint Resistor_SMD:R_0402_1005Metric_Pad0.72x0.64mm_HandSolder -> Resistor_SMD:R_0402_1005Metric
Connections:
- net +3V3: now also J1.1 (Pin_1)
- net FSPI_CS0N: now also J1.2 (Pin_2)
- net FSPI_D0: now also J1.3 (Pin_3)
- net FSPI_D1: now also J1.4 (Pin_4)
- net FSPI_D2: now also J1.5 (Pin_5)
- net FSPI_D3: now also J1.6 (Pin_6)
- net FSPI_SCK: now also J1.7 (Pin_7)
- net GND: now also J1.8 (Pin_8)
- net POGO_RX: no longer names the net of U8.59 (UART0_TX_M0/PWM2_M0/GPIO0_A1_D)
- net POGO_TX: no longer names the net of U8.58 (UART0_RX_M0/CLK_32K/CLK_REFOUT/RTC_CLKO/GPIO0_A0_Z)
Other:
- note added: "SERIAL PORT"
- note removed: "UART0 PORT"
- note removed: "USB-C"
- moved on the sheet: C51, C52, J2, R28, R35, R36, U6

Commit message: feat(Hw):Update_Schematic
Changed lines of the file:
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@@
-		)
-	)
-	(label "D-"
-		(at 119.38 88.9 0)
-		(effects
-			(font
-				(size 1.27 1.27)
-			)
-			(justify left bottom)
 		)
 	)
@@
 	(label "NPOR"
 		(at 269.24 27.94 0)
-		(effects
-			(font
-				(size 1.27 1.27)
-			)
-			(justify left bottom)
-		)
-	)
-	(label "D+"
-		(at 119.38 91.44 0)
 		(effects
 			(font
@@
 		)
 	)
+	(hierarchical_label "D-"
+		(shape input)
+		(at 119.38 88.9 180)
+		(effects
+			(font
+				(size 1.27 1.27)
+			)
+			(justify right)
+		)
+	)
 	(hierarchical_label "MIC-"
 		(shape output)
@@
 		(effects
 			(font
+				(size 1.27 1.27)
+			)
+			(justify right)
+		)
+	)
+	(hierarchical_label "D+"
+		(shape input)
+		(at 119.38 91.44 180)
+		(effects
+			(font

Commit message: feat(Hw):Update_Schematic
Changed lines of the file:
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@@
-		)
-	)
-	(label "USB_DET"
-		(at 119.38 86.36 0)
-		(effects
-			(font
-				(size 1.27 1.27)
-			)
-			(justify left bottom)
 		)
 	)
@@
 		(effects
 			(font
+				(size 1.27 1.27)
+			)
+			(justify right)
+		)
+	)
+	(hierarchical_label "USB_DET"
+		(shape input)
+		(at 119.38 86.36 180)
+		(effects
+			(font

Commit message: feat(Hw):Update_Schematic
Parts:
- removed R34: 22, Resistor_SMD:R_0603_1608Metric, symbol Device:R_Small
- J1: footprint (none) -> Connector_PinHeader_2.54mm:PinHeader_1x08_P2.54mm_Vertical
Connections:
- net GPIO3_C4_D: now reaches U8.2 (VI_CIF_CLKO_M0/MIPI_CLK0_OUT/GPIO3_C4_D)
- net CODEC_MIC1N: now reaches U8.35 (CODEC_MIC1N)
- net CODEC_MIC1P: now reaches U8.36 (CODEC_MIC1P)
- net GPIO4_C1_Z: now reaches U8.22 (SARADC_IN1/PWM1_M1/GPI4_C1_Z)
- net GPIO3_D1_D: now reaches U8.6 (VI_CIF_D13/UART5_RTS_M2/I2C3_SCL_M2/GPIO3_D1_D)
- net GPIO3_D2_D: now reaches U8.8 (VI_CIF_D14/UART5_CTS_M2/I2C3_SDA_M2/GPIO3_D2_D)
- net GPIO3_D3_D: now reaches U8.9 (VI_CIF_D15/PWM1_M2/GPIO3_D3_D)
- net CSI_SCK renamed GPIO3_C7_D
- net CSI_SDA renamed GPIO3_D0_D
- net Lineout renamed CODEC_LINEOUT
- net MCSI_RST renamed GPIO3_C5_D
- net MIC+ renamed CODEC_MIC0P
- net MIC- renamed CODEC_MIC0N
- net MICBIAS renamed CODEC_MICBIAS
- no-connect marks 39 -> 33

Commit message: feat(Hw):Update_Schematic
Connections:
- net GPIO4_A7_U: now reaches U8.38 (EMMC_D5/SPI1_CLK_M0/UART1_RX_M2/I2C2_SCL_M1/GPIO4__A7_U)
- net GPIO4_A5_U: now reaches U8.40 (EMMC_D4/SPI1_CS0_M0/UART1_TX_M2/I2C2_SDA_M1/GPIO4__A5_U)
- net GPIO4_A0_U: now reaches U8.46 (EMMC_D7/SPI1_MISO_M0/UART0_RX_M2/I2C0_SDA_M1/GPIO_4_A0_U)
- net GPIO0_A0_Z: now reaches U8.58 (UART0_RX_M0/CLK_32K/CLK_REFOUT/RTC_CLKO/GPIO0_A0_Z)
- net GPIO0_A1_D: now reaches U8.59 (UART0_TX_M0/PWM2_M0/GPIO0_A1_D)
- net GPIO0_A3_U: now reaches U8.62 (PMIC_PWR_CTRL_M1/GPIO0_A3_U)
- net GPIO1_B0_D: now reaches U8.77 (UART4_RX_M0/PWM3_IR_M1/GPIO1_B0_D)
- net GPIO1_C6_D: now reaches U8.83 (VO_LCDC_D1/VI_CIF_D8_M1/PWM10_M1/UART4_RTS__M1/GPIO1_C6_D)
- net GPIO1_C7_D: now reaches U8.84 (VO_LCDC_D0/VI_CIF_D9_M1/PWM11_IR_M1/UART4_CT_S_M1/GPIO1_C7_D)
- net GPIO1_D2_D: now reaches U8.86 (VO_LCDC_VSYNC/VI_CIF_VSYNC_M1/I2C3_SDA_M1/UA_RT5_RX_M1/SPI0_CS1_M0/PWM0_M1/AUD_DSM_P/GPI_O1_D2_D)
- net GPIO1_D1_D: now reaches U8.87 (VO_LCDC_HSYNC/VI_CIF_HREF_M1/PWM10_M2/UART5__CTS_M1/UART3_RX_M1/GPIO1_D1_D)
- net GPIO1_D0_D: now reaches U8.89 (VO_LCDC_DEN/VI_CIF_CLKI_M1/PWM3_IR_M2/UART5__RTS_M1/UART3_TX_M1/GPIO1_D0_D)
- net GPIO1_C5_D: now reaches U8.90 (VO_LCDC_D2/VI_CIF_D7_M1/PWM9_M1/UART4_TX_M1/_SDMMC1_D2_M1/GPIO1_C5_D)
- net GPIO1_C4_D: now reaches U8.91 (VO_LCDC_D3/VI_CIF_D6_M1/PWM8_M1/UART4_RX_M1_/SDMMC1_D3_M1/GPIO1_C4_D)
- net GPIO1_C3_D: now reaches U8.92 (VO_LCDC_D4/VI_CIF_D5_M1/PWM6_M2/I2C4_SDA_M1/_SDMMC1_CMD_M1/SPI0_MISO_M0/GPIO1_C3_D)
- net GPIO1_C1_D: now reaches U8.94 (VO_LCDC_D6/VI_CIF_D3_M1/PWM4_M2/SPI0_CLK_M0/_SDMMC1_D0_M1/GPIO1_C1_D)
- net GPIO1_C0_D: now reaches U8.95 (VO_LCDC_D7/VI_CIF_D2_M1/PWM2_M2/SPI0_CS0_M0/_SDMMC1_D1_M1/GPIO1_C0_D)
- net ETH_PHY_TXP: now reaches U8.100 (ETH_PHY_TXP)
- net ETH_EXTR: now reaches U8.102 (ETH_EXTR)
- net GPIO2_B1_D_1: now reaches U8.104 (UART0_TX_M1/I2C1_SDA_M1/VO_LCDC_D17/PWM6_M1_/GPIO2_B1_D_1)
- net GPIO2_B1_D_2: now reaches U8.105 (UART0_TX_M1/I2C1_SDA_M1/VO_LCDC_D17/PWM6_M1_/GPIO2_B1_D_2)
- net GPIO2_A7_D: now reaches U8.106 (UART0_CTS_M1/I2S0_SDO1_SDI3/VO_LCDC_D15/PWM_4_M1/I2C3_SDA_M0/PRELIGHT_TRIG_OUT/GPIO2_A7_D)
- net GPIO2_A6_D: now reaches U8.107 (UART0_RTS_M1/I2S0_SDO2_SDI2/VO_LCDC_D14/PWM_2_M1/I2C3_SCL_M0/FLASH_TRIG_OUT/GPIO2_A6_D)
- net GPIO2_A0_D_1: now reaches U8.109 (SDMMC1_D1_M0/I2S0_SCLK/VO_LCDC_D8/UART1_CTS__M1/I2C4_SDA_M0/GPIO2_A0_D_1)
- net GPIO2_A0_D_2: now reaches U8.110 (SDMMC1_D1_M0/I2S0_SCLK/VO_LCDC_D8/UART1_CTS__M1/I2C4_SDA_M0/GPIO2_A0_D_2)
- net GPIO2_A_2_D: now reaches U8.111 (SDMMC1_CLK_M0/I2S0_MCLK/VO_LCDC_D10/GPIO2_A_2_D)
- net GPIO2_A4_D: now reaches U8.113 (SDMMC1_D3_M0/I2S0_SDO0/VO_LCDC_D12/UART1_TX__M1/GPIO2_A4_D)
- net GPIO2_A5_D: now reaches U8.114 (SDMMC1_D2_M0/I2S0_SDI0/VO_LCDC_D13/UART1_RX__M1/GPIO2_A5_D)
- net GPIO3_B2_D: now reaches U8.119 (VI_CIF_D2_M0/MIPI_CSI_RX_CK1N/LVDS_RX_CK1N/GP_IO3_B2_D)
- net GPIO3_B3_D: now reaches U8.120 (VI_CIF_D3_M0/MIPI_CSI_RX_CK1P/LVDS_RX_CK1P/GPI_O3_B3_D)
- net GPIO3_B4_D: now reaches U8.121 (VI_CIF_D4_M0/MIPI_CSI_RX_D2N/LVDS_RX_D2N/GPIO_3_B4_D)
- net GPIO3_B5_D: now reaches U8.122 (VI_CIF_D5_M0/MIPI_CSI_RX_D2P/LVDS_RX_D2P/GPIO3__B5_D)
- net ETH_PHY_RXN: now reaches U8.97 (ETH_PHY_RXN)
- net ETH_PHY_RXP: now reaches U8.98 (ETH_PHY_RXP)
- net ETH_PHY_TXN: now reaches U8.99 (ETH_PHY_TXN)
- net DIN renamed GPIO4_A1_U
- net GPIO renamed GPIO2_A3_D
- net INT renamed GPIO0_A4_D
- net IR_SCL renamed SCL
- net IR_SDA renamed SDA
- net MCSI_CKN renamed GPIO3_C0_D
- net MCSI_CKP renamed GPIO3_C1_D
- net MCSI_D0N renamed GPIO3_C2_D
- net MCSI_D0P renamed GPIO3_C3_D
- net MCSI_D1N renamed GPIO3_B6_D
- net MCSI_D1P renamed GPIO3_B7_D
- net Sound_En renamed GPIO1_D3_D
- no-connect marks 33 -> 0
Other:
- moved on the sheet: R29
