File: hardware/Neopixels.kicad_sch (KiCad schematic)
At the start: 11 parts

Commit message: feat(Hw):Update_Schematic
Parts:
- C2, C21, C43, C46, C47: #LCSC C338117 -> (none); LCSC# (none) -> C338117
- D10, D11, D7, D8, D9: #LCSC C5446700 -> (none); LCSC# (none) -> C5446700
- R4: #LCSC C23179 -> (none); LCSC# (none) -> C23179
Changed lines of the file:
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@@
 			)
 		)
-		(property "#LCSC" "C338117"
-			(at 122.682 54.102 0)
-			(effects
-				(font
-					(size 1.27 1.27)
-				)
+		(property "LCSC#" "C338117"
+			(at 127 54.61 0)
+			(effects
+				(font
+					(size 1.27 1.27)
+				)
+				(hide yes)
 			)
 		)
@@
 			)
 		)
-		(property "#LCSC" "C5446700"
+		(property "LCSC#" "C5446700"
 			(at 82.55 64.77 0)
 			(effects
@@
 			)
 		)
-		(property "#LCSC" "C5446700"
+		(property "LCSC#" "C5446700"
 			(at 102.87 64.77 0)
 			(effects
@@
 			)
 		)
-		(property "#LCSC" "C5446700"
+		(property "LCSC#" "C5446700"
 			(at 124.46 64.77 0)
 			(effects
@@
 			)
 		)
-		(property "#LCSC" "C338117"
-			(at 101.092 54.102 0)
-			(effects
-				(font
-					(size 1.27 1.27)
-				)
+		(property "LCSC#" "C338117"
+			(at 105.41 54.61 0)
+			(effects
+				(font
+					(size 1.27 1.27)
+				)
+				(hide yes)
 			)
 		)
@@
 			)
 		)
-		(property "#LCSC" "C338117"
-			(at 149.352 54.102 0)
-			(effects
-				(font
-					(size 1.27 1.27)
-				)
+		(property "LCSC#" "C338117"
+			(at 153.67 54.61 0)
+			(effects
+				(font
+					(size 1.27 1.27)
+				)
+				(hide yes)
 			)
 		)
@@
 			)
 		)
-		(property "#LCSC" "C338117"
-			(at 80.772 54.102 0)
-			(effects
-				(font
-					(size 1.27 1.27)
-				)
+		(property "LCSC#" "C338117"
+			(at 85.09 54.61 0)
+			(effects
+				(font
+					(size 1.27 1.27)
+				)
+				(hide yes)
 			)
 		)
@@
 			)
 		)
-		(property "#LCSC" "C5446700"
+		(property "LCSC#" "C5446700"
 			(at 151.13 64.77 0)
 			(effects
@@
 			)
 		)
-		(property "#LCSC" "C23179"
+		(property "LCSC#" "C23179"
 			(at 48.26 64.77 90)
 			(effects
@@
 			)
 		)
-		(property "#LCSC" "C5446700"
+		(property "LCSC#" "C5446700"
 			(at 60.96 64.77 0)
 			(effects
@@
 			)
 		)
-		(property "#LCSC" "C338117"
-			(at 59.182 54.102 0)
-			(effects
-				(font
-					(size 1.27 1.27)
-				)
-			)
-		)
+		(property "LCSC#" "C338117"
+			(at 63.5 54.61 0)
+			(effects
+				(font
+					(size 1.27 1.27)
+				)
+				(hide yes)
+			)
+		)

Commit message: feat(Hw):Update_Schematic
Parts:
- D10, D11, D7, D8, D9: footprint pondo:WS2812E-1313 -> Footprints:WS2812E-1313
Changed lines of the file:
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@@
 			)
 		)
-		(property "Footprint" "pondo:WS2812E-1313"
+		(property "Footprint" "Footprints:WS2812E-1313"
 			(at 83.82 72.39 0)
 			(effects
@@
 			)
 		)
-		(property "Footprint" "pondo:WS2812E-1313"
+		(property "Footprint" "Footprints:WS2812E-1313"
 			(at 104.14 72.39 0)
 			(effects
@@
 			)
 		)
-		(property "Footprint" "pondo:WS2812E-1313"
+		(property "Footprint" "Footprints:WS2812E-1313"
 			(at 125.73 72.39 0)
 			(effects
@@
 			)
 		)
-		(property "Footprint" "pondo:WS2812E-1313"
+		(property "Footprint" "Footprints:WS2812E-1313"
 			(at 152.4 72.39 0)
 			(effects
@@
 			)
 		)
-		(property "Footprint" "pondo:WS2812E-1313"
+		(property "Footprint" "Footprints:WS2812E-1313"
 			(at 62.23 72.39 0)
 			(effects
