File: hardware/USB.kicad_sch (KiCad schematic)
At the start: 10 parts, among them J3 USB_A, P4 USB_C_Plug_USB2.0

Commit message: feat(Hw):Update_Schematic
Parts:
- added BT1, BT2, BT3: Battery_Cell, Battery:BatteryHolder_Keystone_2466_1xAAA, symbol Device:Battery_Cell
- added C54: 100nF, Capacitor_SMD:C_0402_1005Metric, symbol Device:C
- added D12: MBR120, Diode_SMD:D_SOD-123F, symbol Diode:MBR340
- added D13: 1N5817, Diode_SMD:D_SOD-123F, symbol Diode:1N5817
- added F2: 750mA, Fuse:Fuse_0603_1608Metric, symbol Device:Fuse_Small
- added Q1: DMG3415U-7, Package_TO_SOT_SMD:SOT-23, symbol Device:Q_PMOS_GSD
- added R11: 100K, Resistor_SMD:R_0603_1608Metric, symbol Device:R_Small
- added R13: 10K, Resistor_SMD:R_0402_1005Metric, symbol Device:R_Small
- added R19: 18k, Resistor_SMD:R_0402_1005Metric, symbol Device:R
- added SW1: ON, FootprintsB:SW-TH_SK12D07VG4, symbol Switch:SW_SPST
- added SW4: SWITCH, symbol Switch:SW_SPDT
- added U1: USB3740B-AI9, symbol Interface_USB:USB3740B-AI9
Connections:
- net +5V: now also SW1.2 (B), SW4.1 (A), U1.5 (VDD); no longer D2.1 (K)
- net D+: now also U1.10 (DP); no longer P4.A6 (D+)
- net D-: now also U1.9 (DM); no longer P4.A7 (D-)
- net GND: now also J3.4 (GND), J3.5 (Shield), BT3.2 (-), C54.2, R11.2, R19.2, SW4.3 (C), U1.3 (OE_N), U1.8 (GND)
- net USB_DET: now also C54.1, R13.1, R19.1
- net at J3.1 (VBUS): now also F2.1
- net 2_DM: now reaches J3.2 (D-)
- net 2_DM: now also U1.7 (DM_2)
- net 2_DP: now reaches J3.3 (D+)
- net 2_DP: now also U1.6 (DP_2)
- new net: BT1.2 (-), BT2.1 (+)
- new net: D12.1 (K), Q1.2 (S), SW1.1 (A)
- new net: D13.2 (A), F2.2, R13.2
- new net: BT2.2 (-), BT3.1 (+)
- new net +BATT: BT1.1 (+), Q1.3 (D)
- new net 1_DM: P4.A7 (D-), U1.1 (DM_1)
- new net 1_DP: P4.A6 (D+), U1.2 (DP_1)
- new net S: SW4.2 (B), U1.4 (S)
- new net VBUS: D12.2 (A), D13.1 (K), D2.1 (K), Q1.1 (G), R11.1
Other:
- note added: "BATTERY"
- note added: "USB-A"
- moved on the sheet: C18, C19, D2, F1, J3, P4, R14, R15, R31, R32

Commit message: feat(Hw):Update_Schematic
Parts:
- removed C19: 100nF, Capacitor_SMD:C_0402_1005Metric, symbol Device:C
- removed R31: 10K, Resistor_SMD:R_0402_1005Metric, symbol Device:R_Small
- removed R32: 18k, Resistor_SMD:R_0402_1005Metric, symbol Device:R
- BT1, BT2, BT3: #LCSC C5290189 -> (none)
Connections:
- net VBUS: now also R13.2
- net at D13.2 (A), F2.2: no longer R13.2
Other:
- moved on the sheet: C54, D13, D2, F1, F2, J3, P4, R13, R14, R15, R19, SW4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

Commit message: feat(Hw):Update_Schematic
Changed lines of the file:
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@@
 	)
 	(hierarchical_label "D-"
-		(shape output)
+		(shape bidirectional)
 		(at 142.24 90.17 0)
 		(effects
@@
 	)
 	(hierarchical_label "D+"
-		(shape output)
+		(shape bidirectional)
 		(at 142.24 87.63 0)
 		(effects

Commit message: feat(Hw):Update_Schematic
Parts:
- added C19, C55: 10uF, symbol Device:C
- added C56, C57: 100uF, symbol Device:C
- added D14, D15: 1N5817, Diode_SMD:D_SOD-123F, symbol Diode:1N5817
- added F3, F4: 750mA, Fuse:Fuse_0603_1608Metric, symbol Device:Fuse_Small
- added J4, J6: USB_A, symbol Connector:USB_A
- added U3: SL2.1A, symbol New_Library:SL2.1A
- added Y5: 12MHz, Crystal:Crystal_SMD_3215-2Pin_3.2x1.5mm, symbol Device:Crystal
Connections:
- net 2_DM: now also U3.9 (UDM)
- net 2_DP: now also U3.10 (UDP)
- net GND: now also C19.1, C55.2, C56.2, C57.2, J4.4 (GND), J4.5 (Shield), J6.4 (GND), J6.5 (Shield), U3.12 (GND)
- net VBUS: now also C56.1, C57.1, D14.1 (K), D15.1 (K), U3.11 (VCC5V)
- new net: C55.1, U3.13 (VDD3)
- new net: C19.2, U3.14 (VDD18)
- new net: D15.2 (A), F4.1
- new net: D14.2 (A), F3.1
- new net: F3.2, J4.1 (VBUS)
- new net: F4.2, J6.1 (VBUS)
- new net 3_DM: J4.2 (D-), U3.7 (DM1)
- new net 3_DP: J4.3 (D+), U3.8 (DP1)
- new net 4_DM: J6.2 (D-), U3.5 (DM2)
- new net 4_DP: J6.3 (D+), U3.6 (DP2)
- new net XIN: U3.16 (XIN), Y5.2
- new net XOUT: U3.15 (XOUT), Y5.1
- no-connect marks 0 -> 4
Other:
- moved on the sheet: C54, D13, D2, F1, F2, J3, P4, R13, R14, R15, R19, SW4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
