File: hardware/Add_On_Bugcon_2025/Add_On_Barrio_del_Hardware.kicad_sch (KiCad schematic)
At the start: 0 parts

Commit message: feat(HW):Init_Sch_PCB
Parts:
- added BT1: Battery_Cell, Add_on:BAT-HLD-001, symbol Device:Battery_Cell
- added C1: 0.1uF, Capacitor_SMD:C_0805_2012Metric, symbol Device:C_Small
- added D2, D3, D4, D5: White, Add_on:LYT77K-K2M1-NoHole, symbol Device:LED_Small
- added D6, D7: Pink, LED_SMD:LED_0603_1608Metric, symbol Device:LED_Small
- added J2: Conn_02x03_Odd_Even, Footprints:B-2100N06P-B111_CKM, symbol Connector_Generic:Conn_02x03_Odd_Even
- added Q1, Q2: 2N7002, Package_TO_SOT_SMD:SOT-23, symbol Transistor_FET:2N7002
- added R2, R3, R4, R5, R8, R9: 180R, Resistor_SMD:R_0805_2012Metric, symbol Device:R_Small
- added R6, R7: 100K, Resistor_SMD:R_0805_2012Metric, symbol Device:R
- added SW1: SW_RST, Button_Switch_SMD:SW_SPST_TL3342, symbol Switch:SW_Push
- added SW2: On, Add_on:MSK12C02, symbol Switch:SW_DPDT_x2
- added U1: PY32F002AL15S6TU, Footprints:PY32F002AL15S6TU, symbol MCU_PY32F002:PY32F002AA15M6TU
Connections:
- new net: D4.1 (K), R4.2
- new net: D7.1 (K), R9.2
- new net: Q1.3 (D), R2.1, R3.1, R8.1
- new net: D3.1 (K), R3.2
- new net: D5.1 (K), R5.2
- new net: D2.1 (K), R2.2
- new net: Q2.3 (D), R4.1, R5.1, R9.1
- new net: BT1.1 (-), SW2.2 (B)
- new net: D6.1 (K), R8.2
- new net +3.3V: BT1.2 (+), C1.1, D2.2 (A), D3.2 (A), D4.2 (A), D5.2 (A), D6.2 (A), D7.2 (A), J2.6 (Pin_6), U1.1 (VCC)
- new net GND: C1.2, J2.5 (Pin_5), Q1.2 (S), Q2.2 (S), R6.2, R7.2, SW1.1, SW2.1 (A), SW2.4 (C), U1.8 (GND)
- new net NRST: SW1.2, U1.6 (PA2/PF2-NRST)
- new net PA1: Q2.1 (G), R7.1, U1.7 (PA1)
- new net PA3: Q1.1 (G), R6.1, U1.3 (PA3)
- new net PA4: U1.2 (PA4/PA10)
- new net SWCLK: J2.2 (Pin_2), U1.4 (PA14-SWC/PB3)
- new net SWDIO: J2.1 (Pin_1), U1.5 (PA13-SWD)
- no-connect marks 0 -> 3
Other:
- note added: "Battery"
- note added: "LED"
- note added: "Microcontroller"
- note added: "RST"
- note added: "Shitty Add-on"

Commit message: feat(Hw):Update_And_Route_PCB
Parts:
- added C2: 0.1uF, Capacitor_SMD:C_0805_2012Metric, symbol Device:C_Small
- D2, D3: LCSC# AA3528SURCKT09 -> (none); manf# (none) -> AA3528SURCKT09
- J2: footprint Footprints:B-2100N06P-B111_CKM -> Connector_PinHeader_2.54mm:PinHeader_2x03_P2.54mm_Vertical_SMD
- R2, R3, R4, R5, R8, R9: value 180R -> 330R; footprint Resistor_SMD:R_0805_2012Metric -> Resistor_SMD:R_0603_1608Metric; LCSC# C1339 -> C105881
- U1: value PY32F002AL15S6TU -> PY32F002AA15M6TU; footprint Footprints:PY32F002AL15S6TU -> Add_on:PY32F002AA15M; LCSC# C5292060 -> C5292058
Connections:
- net PA4 is gone; now on net RX: U1.2 (PF0-OSCIN)
- net GND: now also U1.10 (GND), C2.2; no longer U1.8 (GND)
- net NRST: now also U1.4 (PA0/PF2-NRST), C2.1; no longer U1.6 (PA2/PF2-NRST)
- net PA1: now also Q1.1 (G), R6.1, U1.5 (PA1); no longer Q2.1 (G), R7.1, U1.7 (PA1)
- net SWCLK: now also U1.9 (PA14-SWC/PB3); no longer U1.4 (PA14-SWC/PB3)
- net SWDIO: now also U1.8 (PA13-SWD); no longer U1.5 (PA13-SWD)
- net RX: now reaches J2.3 (Pin_3)
- net TX: now reaches J2.4 (Pin_4)
- net TX: now also U1.3 (PA5/PF1-OSCOUT)
- removed net PA3: Q1.1 (G), R6.1, U1.3 (PA3)
- new net PA6: Q2.1 (G), R7.1, U1.6 (PA6)
- new net PA7: U1.7 (PA7)
- no-connect marks 3 -> 1
Other:
- moved on the sheet: D2, D3, D4, D5, D6, D7, Q1, Q2, R2, R3, R4, R5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

Commit message: feat(Hw)_Update PCB_Hole_Added
Parts:
- added D1: White, LED_SMD:LED_0603_1608Metric, symbol Device:LED_Small
- added R1: 330R, Resistor_SMD:R_0603_1608Metric, symbol Device:R_Small
- D6: value Pink -> Red; LCSC# C7496826 -> C2286
- D7: value Pink -> Green; LCSC# C7496826 -> C916074
Connections:
- net GND: now also R1.1
- net PA7: now also D1.2 (A)
- new net: D1.1 (K), R1.2
