File: hardware/Badge_Bugcon_2025/Badge_Bugcon_2025.kicad_pcb (KiCad board)
At the start: 2 copper layers, 173 parts, among them J1 Conn_01x10_Pin, J1 Flash, J2 Conn_01x04_Pin, J4 Conn_01x03, J5 Conn_Coaxial, P4 USB_C_Plug_USB2.0, Q1 DMG3415U-7, SW2 SW_Push, SW3 SW_Push, U6 W25N02KVZEIR, U7 EA3059, Y1 Crystal, Y2 24MHz, Y3 37.4 Mhz, Y4 OK2EL89CJI-111YLC-32.768K

Commit message: feat(Hw):Init_Floorplan
Parts:
- removed BT1, BT2, BT3: Battery_Cell, Battery:BatteryHolder_Keystone_2466_1xAAA
- removed the C18 at (144.9, 28.7)
- removed the C18 at (115.0, 148.8)
- removed the D2 at (115.0, 147.2)
- removed the D2 at (135.8, 29.4)
- removed the F1 at (116.8, 149.8)
- removed the F1 at (80.2, 27.5)
- removed the J1 at (52.6, 61.2)
- removed the J1 at (155.0, 42.1)
- removed the P4 at (119.2, 154.1)
- removed the P4 at (127.5, 29.9)
- removed the R14 at (118.3, 149.8)
- removed the R14 at (80.2, 35.0)
- removed the R15 at (121.8, 149.8)
- removed the R15 at (80.2, 37.5)
- removed R34: 22, Resistor_SMD:R_0603_1608Metric
- added C18: 10uF, Capacitor_SMD:C_0402_1005Metric, B.Cu at (259.7, 59.2)
- added C55: 10uF, Capacitor_SMD:C_0603_1608Metric, B.Cu at (272.6, 62.0)
- added C56: 100uF, Capacitor_SMD:C_0805_2012Metric, B.Cu at (261.6, 40.3)
- added C57: 100uF, Capacitor_SMD:C_0805_2012Metric, B.Cu at (261.6, 43.4)
- added C66: 0.1uF, Capacitor_SMD:C_0603_1608Metric, B.Cu at (239.4, 78.4)
- added C67: 0.1uF, Capacitor_SMD:C_0603_1608Metric, B.Cu at (239.4, 81.0)
- added C68: 0.1uF, Capacitor_SMD:C_0603_1608Metric, B.Cu at (239.4, 83.5)
- added C69: 0.1uF, Capacitor_SMD:C_0603_1608Metric, B.Cu at (239.4, 86.0)
- added C70: 4.7uF, Capacitor_SMD:C_0603_1608Metric, B.Cu at (272.6, 64.5)
- added C71: 4.7uF, Capacitor_SMD:C_0603_1608Metric, B.Cu at (272.6, 67.0)
- added D14: 1N5817, Diode_SMD:D_SOD-123F, B.Cu at (263.8, 70.0)
- added D15: 1N5817, Diode_SMD:D_SOD-123F, B.Cu at (263.8, 73.3)
- added D16: LED, LED_SMD:LED_0603_1608Metric, B.Cu at (261.4, 30.7)
- added D2: 1N5817, Diode_SMD:D_SOD-123F, B.Cu at (263.8, 59.9)
- added F1: 750mA, Fuse:Fuse_0603_1608Metric, B.Cu at (272.6, 69.5)
- added F3: 750mA, Fuse:Fuse_0603_1608Metric, B.Cu at (268.6, 59.5)
- added F4: 750mA, Fuse:Fuse_0603_1608Metric, B.Cu at (268.6, 62.0)
- added J1: Flash, Connector_PinHeader_2.54mm:PinHeader_1x08_P2.54mm_Vertical, B.Cu at (414.3, -5.67)
- added J3: USB_A, Connector_USB:USB_A_Connfly_DS1095, B.Cu at (114.1, 88.6)
- added J6: USB_A, Connector_USB:USB_A_Connfly_DS1095, B.Cu at (162.0, 106.0)
- added J7: Add_On, Connector_PinSocket_2.54mm:PinSocket_2x03_P2.54mm_Vertical, F.Cu at (47.7, 77.2)
- added J8: OLED, Footprints:Display OLED 128 x32, F.Cu at (120.5, 63.3)
- added J9: Add_On, Connector_PinSocket_2.54mm:PinSocket_2x03_P2.54mm_Vertical, F.Cu at (54.8, 77.2)
- added P4: USB_C_Plug_USB2.0, Footprints:C393939, B.Cu at (107.8, 67.0)
- added R14: 5k1, Resistor_SMD:R_0603_1608Metric, B.Cu at (268.6, 67.0)
- added R15: 5k1, Resistor_SMD:R_0603_1608Metric, B.Cu at (268.6, 69.5)
- added REF**: Batt, Footprints:Batt, B.Cu at (138.1, 102.4)
- added SW4: On, Footprints:MSK12C02, B.Cu at (269.2, 43.7)
- added SW5: SW_Push, Button_Switch_SMD:SW_SPST_TL3342, F.Cu at (38.0, 78.4)
- added SW6: SW_Push, Button_Switch_SMD:SW_SPST_TL3342, F.Cu at (38.0, 85.4)
- added SW7: SW_Push, Button_Switch_SMD:SW_SPST_TL3342, F.Cu at (38.0, 92.5)
- added SW8: SW_Push, Button_Switch_SMD:SW_SPST_TL3342, F.Cu at (38.0, 99.5)
- added U1: USB3740B-AI9, Package_DFN_QFN:UQFN-10_1.3x1.8mm_P0.4mm, B.Cu at (259.4, 53.3)
- added U2: AP6256, Footprints:XCVR_AP6255, B.Cu at (408.5, 101.8)
- added U3: SL2.1A, Package_SO:SOP-16_3.9x9.9mm_P1.27mm, B.Cu at (270.4, 52.5)
- added U5: MCP73831T-2ATI/OT, Package_TO_SOT_SMD:SOT-23-5, B.Cu at (263.5, 49.0)
- added Y5: 12MHz, Crystal:Crystal_SMD_3225-4Pin_3.2x2.5mm, B.Cu at (272.0, 75.6)
- C1, C10, C11, C12, C13, C14, C15, C16, C17, C2, C20, C21, C22, C23, C24, C25, C26, C27, C28, C29, C3, C30, C31, C32, C33, C34, C35, C36, C37, C38, C39, C4, C40, C41, C42, C43, C44, C45, C46, C47, C48, C49, C5, C50, C51, C52, C53, C54, C58, C59, C6, C60, C61, C62, C63, C64, C65, C7, C8, C86, C9, D1, D10, D11, D12, D13, D3, D4, D5, D6, D7, D8, D9, F2, FB1, FB2, FB3, J2, J5, L1, L4, L5, L6, L7, Q1, R1, R10, R11, R12, R13, R16, R17, R18, R19, R2, R20, R21, R22, R23, R24, R25, R26, R27, R28, R29, R3, R30, R33, R35, R36, R38, R39, R4, R41, R42, R43, R44, R45, R46, R47, R48, R49, R5, R50, R52, R53, R54, R55, R56, R57, R58, R59, R6, R60, R61, R62, R63, R64, R7, R8, R9, SW2, SW3, U4, U6, U7, U8, Y1, Y2, Y3, Y4: moved to B.Cu
- C19: value 100nF -> 10uF; footprint Capacitor_SMD:C_0402_1005Metric_Pad0.74x0.62mm_HandSolder -> Capacitor_SMD:C_0603_1608Metric; moved to B.Cu
- J4: value Conn_01x03 -> USB_A; footprint Connector_PinHeader_2.54mm:PinHeader_1x03_P2.54mm_Vertical -> Connector_USB:USB_A_Connfly_DS1095; moved to B.Cu
- R31: value 10K -> 2k; footprint Resistor_SMD:R_0402_1005Metric_Pad0.72x0.64mm_HandSolder -> LED_SMD:LED_0603_1608Metric; moved to B.Cu
- R32: value 18k -> 470; footprint Resistor_SMD:R_0402_1005Metric_Pad0.72x0.64mm_HandSolder -> LED_SMD:LED_0603_1608Metric; moved to B.Cu
- moved R39 460.8 mm to (487.9, 175.5), turned to 180 degrees
- moved R41 460.8 mm to (487.9, 178.0), turned to 180 degrees
- moved R42 460.8 mm to (487.9, 180.5), turned to 180 degrees
- moved R43 460.8 mm to (487.9, 183.0), turned to 180 degrees
- moved C11 454.5 mm to (470.2, 162.2)
- moved C12 454.1 mm to (470.2, 161.3)
- moved R6 444.2 mm to (470.2, 163.2)
- moved L6 444.0 mm to (467.0, 162.2)
- moved R21 440.8 mm to (470.2, 164.1)
- moved C59 436.9 mm to (462.5, 171.2), turned to -90 degrees
- moved L5 436.5 mm to (467.2, 170.2)
- moved C58 435.2 mm to (462.7, 161.1), turned to 90 degrees
- moved C86 434.3 mm to (461.0, 171.2), turned to -90 degrees
- moved C9 433.5 mm to (470.5, 169.2)
- moved C10 433.5 mm to (470.5, 171.1)
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Connections:
- net Net-(U8D-ETH_AVDD3V3) renamed /MCU/ETH_AVDD3V3
- C19 pad 1: /MCU/USB_DET -> GND
- C19 pad 2: GND -> Net-(U3-VDD18)
- J4 pad 1: GND -> Net-(J4-VBUS)
- J4 pad 2: /MCU/GPIO -> /USB/3_DM
- J4 pad 3: +3V3 -> /USB/3_DP
- R31 pad 1: /MCU/USB_DET -> Net-(U5-PROG)
- R31 pad 2: Net-(D2-A) -> GND
- R32 pad 1: /MCU/USB_DET -> Net-(D16-K)
- R32 pad 2: GND -> /USB/STAT
- U8 pad 58: /MCU/GPIO0_A0_Z -> /MCU/LEFT
- U8 pad 59: /MCU/GPIO0_A1_D -> /MCU/RIGHT
- U8 pad 62: /MCU/GPIO0_A3_U -> /MCU/DOWN
- U8 pad 63: /MCU/GPIO0_A4_D -> /MCU/UP
- U8 pad 72: /MCU/GPIO1_A0_D -> /MCU/SCL
- U8 pad 73: /MCU/GPIO1_A1_D -> /MCU/SDA
Other:
- board outline added: 100 x 100 mm

Commit message: feat(Hw):Update_Schematic_And_Floorplan
Parts:
- removed REF**: Batt, Footprints:Batt
- added J10: Battery, Footprints:Batt, B.Cu at (138.4, 102.0)
- added J11: +1V8, Connector_PinHeader_2.54mm:PinHeader_1x20_P2.54mm_Vertical, F.Cu at (-32.1, 31.0)
- added J12: CODEC, Connector_PinHeader_2.54mm:PinHeader_1x08_P2.54mm_Vertical, F.Cu at (-27.5, 31.0)
- added J13: ETH, Connector_PinHeader_2.54mm:PinHeader_1x07_P2.54mm_Vertical, F.Cu at (-27.5, 53.3)
- added J14: +3V3, Connector_PinHeader_2.54mm:PinHeader_1x28_P2.54mm_Vertical, F.Cu at (-40.9, 25.2)
- added SW1: ON, Button_Switch_THT:SW_Slide_SPDT_Angled_CK_OS102011MA1Q, F.Cu at (314.0, 52.0)
- C1, C2, C21, C24, C28, C34, C38, C43, C46, C47, C48, C51, C62, C64: footprint Capacitor_SMD:C_0603_1608Metric -> Capacitor_SMD:C_0402_1005Metric
- C66, C67, C68, C69: moved to F.Cu
- R16, R17, R25, R27, R3, R39: footprint Resistor_SMD:R_0603_1608Metric -> Resistor_SMD:R_0402_1005Metric
- moved C2 220.9 mm to (48.0, 39.9)
- moved C21 220.8 mm to (48.0, 42.9)
- moved C43 220.7 mm to (48.0, 45.9)
- moved C46 220.6 mm to (48.0, 48.9)
- moved C47 220.5 mm to (48.0, 51.9)
- moved D10 216.8 mm to (48.0, 50.2)
- moved D11 216.8 mm to (48.0, 53.2)
- moved D7 216.8 mm to (48.0, 41.1)
- moved D8 216.8 mm to (48.0, 44.1)
- moved D9 216.8 mm to (48.0, 47.2)
- moved R4 216.8 mm to (51.9, 53.5)
- moved C19 195.2 mm to (106.3, 161.8), turned to 0 degrees
- moved C55 194.7 mm to (106.3, 163.3)
- moved U3 191.1 mm to (114.3, 162.8)
- moved Y5 185.7 mm to (106.1, 159.0), turned to 90 degrees
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Connections:
- Y5 pad 2: /USB/XIN -> (no net)
- Y5 pad 3: (no net) -> /USB/XIN

Commit message: feat(Hw):Update_Schematic
Parts:
- added R34: 6K, Resistor_SMD:R_0805_2012Metric, B.Cu at (427.4, -24.1)
- C22, C31, C32, C33, C44, C50, C53: footprint Capacitor_SMD:C_0402_1005Metric_Pad0.74x0.62mm_HandSolder -> Capacitor_SMD:C_0402_1005Metric
- C37: footprint Capacitor_SMD:C_0603_1608Metric_Pad1.08x0.95mm_HandSolder -> Capacitor_SMD:C_0603_1608Metric
- R39: value 100 -> 330
- R44, R45, R46, R47, R48, R49, R50, R52, R53, R54, R55, R56, R57, R58, R59, R60, R61, R62, R63, R64: footprint Resistor_SMD:R_0402_1005Metric_Pad0.72x0.64mm_HandSolder -> Resistor_SMD:R_0402_1005Metric

Commit message: feat(Hw):Update_Schematic_And_Floorplan
Parts:
- removed C22, C31: 22uf, Capacitor_SMD:C_0402_1005Metric
- removed C32, C33: 14pf, Capacitor_SMD:C_0402_1005Metric
- removed C37: 4.7uf, Capacitor_SMD:C_0603_1608Metric
- removed C44: 15pf, Capacitor_SMD:C_0402_1005Metric
- removed C45: 10uF, Capacitor_SMD:C_0603_1608Metric
- removed C50, C53: 100nF, Capacitor_SMD:C_0402_1005Metric
- removed FB3: BLM21PG121SN1D, Inductor_SMD:L_0805_2012Metric
- removed L1: 1uH, Inductor_SMD:L_1008_2520Metric
- removed R44, R59: 4.7K, Resistor_SMD:R_0402_1005Metric
- removed R45, R46, R47, R48, R49, R52, R53, R54, R56, R57, R58, R61, R62, R63, R64: 10K, Resistor_SMD:R_0402_1005Metric
- removed R50: 100K, Resistor_SMD:R_0402_1005Metric
- removed R55, R60: 1K, Resistor_SMD:R_0402_1005Metric
- removed U2: AP6256, Footprints:XCVR_AP6255
- removed U4: ~, Package_TO_SOT_SMD:SuperSOT-6
- removed Y3: 37.4 Mhz, Footprints:SMD1612-4P
- removed Y4: OK2EL89CJI-111YLC-32.768K, Crystal:Crystal_SMD_3225-4Pin_3.2x2.5mm
- added J2: Conn_01x04, Connector_PinHeader_2.54mm:PinHeader_1x04_P2.54mm_Vertical, F.Cu at (-94.0, 34.5)
- J11: value +1V8 -> +3V3; footprint Connector_PinHeader_2.54mm:PinHeader_1x20_P2.54mm_Vertical -> Connector_PinHeader_2.54mm:PinHeader_1x21_P2.54mm_Vertical
- J14: value +3V3 -> +1V8; footprint Connector_PinHeader_2.54mm:PinHeader_1x28_P2.54mm_Vertical -> Connector_PinHeader_2.54mm:PinHeader_1x23_P2.54mm_Vertical
- J5: value Conn_Coaxial -> +3V3; footprint Connector_Coaxial:U.FL_Molex_MCRF_73412-0110_Vertical -> Connector_PinHeader_2.54mm:PinHeader_1x22_P2.54mm_Vertical; moved to F.Cu
- moved J5 487.4 mm to (-103.2, 34.5), turned to 0 degrees
- moved J14 67.6 mm to (-107.8, 34.5)
- moved J11 66.6 mm to (-98.6, 34.5)
- moved J12 64.2 mm to (-87.6, 53.5)
- moved J13 55.5 mm to (-83.0, 53.5)
Connections:
- C71 pad 1: Net-(U5-V_{BAT}) -> +BATT
- J11 pad 1: +1V8 -> +3V3
- J11 pad 10: /MCU/GPIO3_B3_D -> /MCU/GPIO1_C0_D
- J11 pad 11: /MCU/GPIO3_B4_D -> /MCU/GPIO2_B1_D_1
- J11 pad 12: /MCU/GPIO3_B5_D -> /MCU/GPIO2_B1_D_2
- J11 pad 13: /MCU/GPIO3_B6_D -> /MCU/GPIO2_A7_D
- J11 pad 14: /MCU/GPIO3_B7_D -> /MCU/GPIO2_A6_D
- J11 pad 15: /MCU/GPIO3_C0_D -> /MCU/GPIO2_A0_D_1
- J11 pad 16: /MCU/GPIO3_C1_D -> /MCU/GPIO2_A0_D_2
- J11 pad 17: /MCU/GPIO3_C2_D -> /MCU/GPIO2_A_2_D
- J11 pad 18: /MCU/GPIO3_C3_D -> /MCU/GPIO2_A3_D
- J11 pad 19: /MCU/GPIO4_C1_Z -> /MCU/GPIO2_A4_D
- J11 pad 2: /MCU/GPIO3_C4_D -> /MCU/GPIO1_D3_D
- J11 pad 20: GND -> /MCU/GPIO2_A5_D
- J11 pad 3: /MCU/GPIO3_C5_D -> /MCU/GPIO1_D2_D
- J11 pad 4: /MCU/GPIO3_C7_D -> /MCU/GPIO1_D1_D
- J11 pad 5: /MCU/GPIO3_D1_D -> /MCU/GPIO1_D0_D
- J11 pad 6: /MCU/GPIO3_D0_D -> /MCU/GPIO1_C5_D
- J11 pad 7: /MCU/GPIO3_D2_D -> /MCU/GPIO1_C4_D
- J11 pad 8: /MCU/GPIO3_D3_D -> /MCU/GPIO1_C3_D
- J11 pad 9: /MCU/GPIO3_B2_D -> /MCU/GPIO1_C1_D
- J14 pad 1: +3V3 -> +1V8
- J14 pad 10: /MCU/GPIO1_D2_D -> /MCU/GPIO4_C1_Z
- J14 pad 11: /MCU/GPIO1_D1_D -> /MCU/GPIO3_B0_D
- J14 pad 12: /MCU/GPIO1_D0_D -> /MCU/GPIO3_B1_D
- J14 pad 13: /MCU/GPIO1_C5_D -> /MCU/GPIO3_B2_D
- J14 pad 14: /MCU/GPIO1_C4_D -> /MCU/GPIO3_B3_D
- J14 pad 15: /MCU/GPIO1_C3_D -> /MCU/GPIO3_B4_D
- J14 pad 16: /MCU/GPIO1_C1_D -> /MCU/GPIO3_B5_D
- J14 pad 17: /MCU/GPIO1_C0_D -> /MCU/GPIO3_B6_D
- J14 pad 18: /MCU/GPIO2_B1_D_1 -> /MCU/GPIO3_B7_D
- J14 pad 19: /MCU/GPIO2_B1_D_2 -> /MCU/GPIO3_C0_D
- J14 pad 2: /MCU/GPIO4_A7_U -> /MCU/GPIO3_C4_D
- J14 pad 20: /MCU/GPIO2_A7_D -> /MCU/GPIO3_C1_D
- J14 pad 21: /MCU/GPIO2_A6_D -> /MCU/GPIO3_C2_D
- J14 pad 22: /MCU/GPIO2_A0_D_1 -> /MCU/GPIO3_C3_D
- J14 pad 23: /MCU/GPIO2_A0_D_2 -> GND
- J14 pad 3: /MCU/GPIO4_A5_U -> /MCU/GPIO3_C5_D
- J14 pad 4: /MCU/GPIO4_A1_U -> /MCU/LED
- J14 pad 5: /MCU/GPIO4_A0_U -> /MCU/GPIO3_C7_D
- J14 pad 6: /MCU/GPIO1_B0_D -> /MCU/GPIO3_D1_D
- J14 pad 7: /MCU/GPIO1_C6_D -> /MCU/GPIO3_D0_D
- J14 pad 8: /MCU/GPIO1_C7_D -> /MCU/GPIO3_D2_D
- J14 pad 9: /MCU/GPIO1_D3_D -> /MCU/GPIO3_D3_D
- J5 pad 1: /Wifi_Module/AP6256_ANTENNA -> +3V3
- J5 pad 2: GND -> /MCU/GPIO3_A2_U
- U5 pad 3: Net-(U5-V_{BAT}) -> +BATT
- U8 pad 117: /MCU/BT_HOST_WAKE -> /MCU/GPIO3_B0_D
- U8 pad 118: /MCU/WT_HOST_WAKE -> /MCU/GPIO3_B1_D
- U8 pad 12: /MCU/DAT1_SDIO -> /MCU/GPIO3_A2_U
- U8 pad 14: /MCU/DAT0_SDIO -> /MCU/GPIO3_A3_U
- U8 pad 15: /MCU/CLK_SDIO -> /MCU/GPIO3_A4_D
- U8 pad 16: /MCU/CMD_SDIO -> /MCU/GPIO3_A5_U
- U8 pad 17: /MCU/DAT3_SDIO -> /MCU/GPIO3_A6_U
- U8 pad 18: /MCU/DAT2_SDIO -> /MCU/GPIO3_A7_U
- U8 pad 60: /MCU/BT_WAKE -> /MCU/GPIO0_A2_D
- U8 pad 64: /MCU/CTS_BT -> /MCU/GPIO0_A5_D
- U8 pad 65: /MCU/RTS_BT -> /MCU/GPIO0_A6_D
- U8 pad 74: /Wifi_Module/WL_EN -> /MCU/GPIO1_A2_D
- U8 pad 75: /MCU/TX_BT -> /MCU/GPIO1_A3_D
- U8 pad 76: /MCU/RX_BT -> /MCU/GPIO1_A4_D
- U8 pad 78: /MCU/BT_REG_ON -> /MCU/GPIO1_B1_D

Commit message: feat(Hw):Update_Schematic_And_Floorplan
Parts:
- removed C21, C43, C46, C47: 100nF, Capacitor_SMD:C_0402_1005Metric
- removed C66, C67, C68, C69: 0.1uF, Capacitor_SMD:C_0603_1608Metric
- removed D10, D11, D9: WS2812E-1313, Footprints:WS2812E-1313
- removed J11: +3V3, Connector_PinHeader_2.54mm:PinHeader_1x21_P2.54mm_Vertical
- removed the J2 at (-94.0, 34.5)
- removed the J2 at (228.1, 45.4)
- removed SW5, SW6, SW7, SW8: SW_Push, Button_Switch_SMD:SW_SPST_TL3342
- removed U5: MCP73831T-2ATI/OT, Package_TO_SOT_SMD:SOT-23-5
- added J2: Conn_01x04, Connector_PinHeader_2.54mm:PinHeader_1x04_P2.54mm_Vertical, F.Cu at (414.9, -125.9)
- added U2: TP4056, Package_SO:SOIC-8-1EP_3.9x4.9mm_P1.27mm_EP2.41x3.3mm_ThermalVias, B.Cu at (320.0, 32.5)
- C70, C71: value 4.7uF -> 10uF
- D8: value WS2812E-1313 -> LED; footprint Footprints:WS2812E-1313 -> LED_SMD:LED_0603_1608Metric
- J10: footprint Footprints:Batt -> Battery:BatteryHolder_Keystone_1042_1x18650
- J5: value +3V3 -> 3V3; footprint Connector_PinHeader_2.54mm:PinHeader_1x22_P2.54mm_Vertical -> Connector_PinSocket_2.54mm:PinSocket_1x24_P2.54mm_Vertical
- J8: value OLED -> 3V3; footprint Footprints:Display OLED 128 x32 -> Connector_PinSocket_2.54mm:PinSocket_1x23_P2.54mm_Vertical
- R31: footprint LED_SMD:LED_0603_1608Metric -> Resistor_SMD:R_0603_1608Metric
- R32: value 470 -> 10K; footprint LED_SMD:LED_0603_1608Metric -> Resistor_SMD:R_0402_1005Metric
- moved J5 562.4 mm to (421.1, -169.0)
- moved J14 556.3 mm to (410.3, -168.2)
- moved J12 549.2 mm to (414.9, -168.2)
- moved J13 536.3 mm to (414.9, -145.8)
- moved J8 383.5 mm to (425.7, -169.0)
- moved D8 266.2 mm to (313.9, 33.3)
- moved J10 177.2 mm to (3.83, -13.2), turned to 0 degrees
- moved C70 22.3 mm to (313.9, 29.0)
- moved R32 22.0 mm to (324.8, 31.9), turned to 0 degrees
- moved R31 20.4 mm to (313.9, 30.4)
- moved R4 14.5 mm to (45.0, 40.7), turned to 0 degrees
- moved C71 12.3 mm to (313.9, 34.8), turned to 180 degrees
- moved D16 11.9 mm to (313.9, 31.9)
- moved C54 11.9 mm to (259.6, 24.8)
- moved R13 11.9 mm to (259.6, 22.9)
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Connections:
- D16 pad 2: VBUS -> Net-(D16-A)
- D7 pad 2: Net-(D7-DOUT) -> unconnected-(D7-DOUT-Pad2)
- D8 pad 1: +3V3 -> Net-(D8-K)
- D8 pad 2: Net-(D8-DOUT) -> Net-(D16-A)
- J12 pad 1: /MCU/VCC1V8_CODEC -> +1V8
- J5 pad 12: /MCU/GPIO0_A2_D -> /MCU/GPIO0_A0_Z
- J5 pad 13: /MCU/GPIO0_A5_D -> /MCU/GPIO0_A1_D
- J5 pad 14: /MCU/GPIO0_A6_D -> /MCU/GPIO0_A2_D
- J5 pad 15: /MCU/GPIO1_A2_D -> /MCU/GPIO0_A3_U
- J5 pad 16: /MCU/GPIO1_A3_D -> /MCU/GPIO0_A4_D
- J5 pad 17: /MCU/GPIO1_A4_D -> /MCU/GPIO0_A5_D
- J5 pad 18: /MCU/GPIO1_B0_D -> /MCU/GPIO0_A6_D
- J5 pad 19: /MCU/GPIO1_B1_D -> /MCU/GPIO1_A2_D
- J5 pad 20: /MCU/GPIO1_C6_D -> /MCU/GPIO1_A3_D
- J5 pad 21: /MCU/GPIO1_C7_D -> /MCU/GPIO1_A4_D
- J5 pad 22: GND -> /MCU/GPIO1_B0_D
- J7 pad 3: /MCU/SDA -> /Add-On/SDA
- J7 pad 4: /MCU/SCL -> /Add-On/SCL
- J8 pad 1: /MCU/SDA -> +3V3
- J8 pad 2: /MCU/SCL -> /MCU/GPIO1_C6_D
- J8 pad 3: +3V3 -> /MCU/GPIO1_C7_D
- J8 pad 4: GND -> /MCU/GPIO1_D3_D
- J9 pad 3: /MCU/SDA -> /Add-On/SDA
- J9 pad 4: /MCU/SCL -> /Add-On/SCL
- R31 pad 1: Net-(U5-PROG) -> VBUS
- R31 pad 2: GND -> Net-(D16-A)
- R32 pad 1: Net-(D16-K) -> Net-(U2-PROG)
- R32 pad 2: /USB/STAT -> GND
- U8 pad 58: /MCU/LEFT -> /MCU/GPIO0_A0_Z
- U8 pad 59: /MCU/RIGHT -> /MCU/GPIO0_A1_D
- U8 pad 62: /MCU/DOWN -> /MCU/GPIO0_A3_U
- U8 pad 63: /MCU/UP -> /MCU/GPIO0_A4_D
- U8 pad 72: /MCU/SCL -> /Add-On/SCL
- U8 pad 73: /MCU/SDA -> /Add-On/SDA

Commit message: feat(Hw):Update_Schematic_And_Floorplan
Parts:
- C1, C2, C20, C23, C24, C25, C26, C27, C28, C29, C3, C30, C34, C35, C36, C38, C39, C4, C40, C41, C42, C48, C49, C5, C51, C52, C6, C60, C62, C63, C64, C65, D1, D7, FB1, FB2, J1, R10, R16, R17, R18, R2, R25, R26, R27, R28, R29, R3, R30, R33, R34, R35, R36, R4, R9, SW2, SW3, U6, U8, Y1, Y2: moved to F.Cu
- J10: footprint Battery:BatteryHolder_Keystone_1042_1x18650 -> Footprints:BatteryHolder_Keystone_1042_1x18650
- R31: value 2k -> 2K
- R32: value 10K -> 2K; footprint Resistor_SMD:R_0402_1005Metric -> Resistor_SMD:R_0603_1608Metric
- SW1: moved to B.Cu
- moved J8 389.4 mm to (113.0, 63.1), turned to 90 degrees
- moved J12 384.7 mm to (113.0, 70.2), turned to 90 degrees
- moved J5 383.6 mm to (113.0, 59.5), turned to 90 degrees
- moved J14 378.9 mm to (113.0, 66.7), turned to 90 degrees
- moved J13 354.1 mm to (134.3, 70.3), turned to 90 degrees
- moved J1 352.2 mm to (127.8, 120.5), turned to 90 degrees
- moved C20 347.1 mm to (118.1, 96.5)
- moved Y1 342.4 mm to (120.6, 96.2), turned to 0 degrees
- moved FB1 341.4 mm to (121.1, 104.7), turned to 0 degrees
- moved R16 340.3 mm to (123.7, 108.8), turned to 180 degrees
- moved C62 340.3 mm to (121.7, 102.6), turned to 180 degrees
- moved C63 340.3 mm to (121.7, 103.5), turned to 180 degrees
- moved D1 339.8 mm to (121.9, 88.5), turned to 0 degrees
- moved R3 339.8 mm to (121.9, 89.8), turned to 180 degrees
- moved R35 339.2 mm to (124.2, 110.0), turned to 180 degrees
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Connections:
- net +5V renamed VCC
Other:
- outline, holes or cut-outs redrawn

Commit message: feat(Hw):Update_Floorplan
Parts:
- C54, R13, R19, SW1, SW4: moved to F.Cu
- moved R13 158.3 mm to (123.1, 102.9), turned to 0 degrees
- moved R19 158.3 mm to (123.1, 103.9), turned to 0 degrees
- moved C54 158.3 mm to (123.1, 104.8), turned to 0 degrees
- moved U1 157.9 mm to (105.2, 101.5), turned to 90 degrees
- moved SW4 144.7 mm to (102.3, 78.5), turned to -90 degrees
- moved R39 130.9 mm to (136.0, 77.7)
- moved R41 130.9 mm to (136.0, 80.2)
- moved R42 130.9 mm to (136.0, 82.7)
- moved R43 130.9 mm to (136.0, 85.2)
- moved D3 124.9 mm to (132.3, 77.8)
- moved D4 124.9 mm to (132.3, 80.4)
- moved D5 124.9 mm to (132.3, 82.9)
- moved D6 124.9 mm to (132.3, 85.5)
- moved C13 124.3 mm to (124.8, 80.4)
- moved C14 124.3 mm to (124.8, 79.5)
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Connections:
- J3 pad 2: /USB/2_DM -> /USB/1_DM
- J3 pad 3: /USB/2_DP -> /USB/1_DP
- P4 pad A6: /USB/1_DP -> /USB/2_DP
- P4 pad A7: /USB/1_DM -> /USB/2_DM
- U3 pad 10: /USB/2_DP -> /USB/1_DP
- U3 pad 9: /USB/2_DM -> /USB/1_DM

Commit message: feat(Hw):Updated_Floorplan
Parts:
- moved J5 68.4 mm to (106.4, 127.6)
- moved J12 63.6 mm to (146.9, 124.0)
- moved J8 58.7 mm to (171.7, 62.7), turned to -90 degrees
- moved R43 34.2 mm to (105.7, 69.6), turned to 0 degrees
- moved R42 32.2 mm to (105.7, 72.1), turned to 0 degrees
- moved R41 30.9 mm to (105.7, 74.6), turned to 0 degrees
- moved R39 30.4 mm to (105.7, 77.1), turned to 0 degrees
- moved D6 28.1 mm to (109.4, 69.3), turned to 0 degrees
- moved D5 25.4 mm to (109.4, 71.9), turned to 0 degrees
- moved D4 23.7 mm to (109.4, 74.5), turned to 0 degrees
- moved D3 22.9 mm to (109.4, 77.1), turned to 0 degrees
- moved C57 8.66 mm to (166.8, 79.8), turned to -90 degrees
- moved F4 8.60 mm to (171.1, 79.5), turned to 90 degrees
- moved D15 7.98 mm to (169.0, 80.2), turned to 90 degrees
- moved C70 7.60 mm to (165.0, 75.6)
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