File: hardware/Badge_Bugcon_2025/Badge_Bugcon_2025.kicad_pcb (KiCad board)
At the start: 2 copper layers, 100 x 100 mm, 147 parts, among them J1 Flash, J10 Battery, J12 CODEC, J13 ETH, J14 +1V8, J2 Conn_01x04, J3 USB_A, J4 USB_A, J5 3V3, J6 USB_A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

Commit message: feat(Hw):Init_Route
Parts:
- removed J12: CODEC, Connector_PinHeader_2.54mm:PinHeader_1x08_P2.54mm_Vertical
- removed J2: Conn_01x04, Connector_PinHeader_2.54mm:PinHeader_1x04_P2.54mm_Vertical
- J1: value Flash -> Conn_01x21; footprint Connector_PinHeader_2.54mm:PinHeader_1x08_P2.54mm_Vertical -> Connector_PinHeader_2.54mm:PinHeader_1x21_P2.54mm_Vertical
- moved R42 24.1 mm to (127.7, 81.8), turned to 180 degrees
- moved R41 22.2 mm to (127.6, 71.2), turned to 180 degrees
- moved D4 20.3 mm to (127.7, 83.2)
- moved D5 18.4 mm to (127.6, 69.7)
- moved J13 16.1 mm to (150.4, 69.4), turned to -90 degrees
- moved C15 12.1 mm to (116.0, 81.0), turned to -90 degrees
- moved J1 9.39 mm to (116.1, 124.0)
- moved R39 6.20 mm to (109.8, 81.7)
- moved D3 5.95 mm to (110.3, 82.9), turned to 180 degrees
- moved J5 5.94 mm to (112.3, 127.5)
- moved R6 5.50 mm to (124.4, 74.1), turned to -90 degrees
- moved C9 5.38 mm to (124.5, 78.7), turned to 90 degrees
- moved C56 5.12 mm to (165.6, 104.9), turned to 180 degrees
- moved C11 5.01 mm to (125.3, 74.1), turned to -90 degrees
- moved R43 4.99 mm to (110.2, 71.6)
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Connections:
- net /USB/1_DM renamed /USB/1_DN
- net /USB/2_DM renamed /USB/2_DN
- net /USB/3_DM renamed /USB/3_DN
- net /USB/4_DM renamed /USB/4_DN
- J1 pad 1: +3V3 -> +1V8
- J1 pad 2: /MCU/FSPI_CS0N -> /MCU/CODEC_LINEOUT
- J1 pad 3: /MCU/FSPI_D0 -> /MCU/CODEC_MICBIAS
- J1 pad 4: /MCU/FSPI_D1 -> /MCU/CODEC_MIC0N
- J1 pad 5: /MCU/FSPI_D2 -> /MCU/CODEC_MIC0P
- J1 pad 6: /MCU/FSPI_D3 -> /MCU/CODEC_MIC1N
- J1 pad 7: /MCU/FSPI_SCK -> /MCU/CODEC_MIC1P
- J14 pad 10: /MCU/GPIO4_C1_Z -> /MCU/GPIO3_C4_D
- J14 pad 2: /MCU/GPIO3_C4_D -> /MCU/GPIO4_C1_Z
- J14 pad 3: /MCU/GPIO3_C5_D -> /MCU/GPIO3_D3_D
- J14 pad 4: /MCU/LED -> /MCU/GPIO3_D2_D
- J14 pad 5: /MCU/GPIO3_C7_D -> /MCU/GPIO3_D0_D
- J14 pad 7: /MCU/GPIO3_D0_D -> /MCU/GPIO3_C7_D
- J14 pad 8: /MCU/GPIO3_D2_D -> /MCU/LED
- J14 pad 9: /MCU/GPIO3_D3_D -> /MCU/GPIO3_C5_D
Routing:
- net /USB/1_DP: track 0.00 -> 48.5 mm, vias 0 -> 1
- net /USB/1_DN: track 0.00 -> 47.7 mm, vias 0 -> 1
- net /USB/4_DN: track 0.00 -> 46.1 mm
- net /USB/4_DP: track 0.00 -> 46.1 mm
- net /MCU/FSPI_D0: track 0.00 -> 29.2 mm
- net /MCU/FSPI_D2: track 0.00 -> 27.8 mm
- net /USB/3_DN: track 0.00 -> 27.1 mm
- net /USB/3_DP: track 0.00 -> 27.1 mm
- net /MCU/FSPI_SCK: track 0.00 -> 26.1 mm
- net /MCU/D-: track 0.00 -> 25.3 mm, vias 0 -> 1
- net /MCU/D+: track 0.00 -> 25.3 mm, vias 0 -> 1
- net /MCU/FSPI_D1: track 0.00 -> 23.9 mm
- net /MCU/FSPI_D3: track 0.00 -> 22.1 mm
- net /MCU/FSPI_CS0N: track 0.00 -> 20.0 mm
- net VCC: track 0.00 -> 17.2 mm
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- added copper zone on B.Cu, net +1V8
- added copper zone on B.Cu, net +3V3
- added copper zone on B.Cu, net /Buck_Converter/VCC_DDR
- added copper zone on B.Cu, net /Buck_Converter/v_0.9v

Commit message: feat(Hw):Update_Route
Parts:
- moved C38 12.8 mm to (145.5, 99.0), turned to 0 degrees
- moved Y5 12.4 mm to (145.8, 107.4)
- moved C55 12.4 mm to (146.0, 111.7)
- moved C19 12.4 mm to (146.0, 110.2)
- moved U3 12.4 mm to (152.8, 111.2)
- moved R16 10.1 mm to (137.2, 111.5), turned to 90 degrees
- moved C52 9.42 mm to (137.1, 115.4)
- moved R35 9.42 mm to (136.6, 113.6)
- moved C51 9.42 mm to (136.1, 115.4)
- moved R36 9.42 mm to (148.2, 111.8)
- moved U6 9.42 mm to (142.6, 113.0)
- moved F4 8.55 mm to (166.7, 85.4)
- moved C57 8.05 mm to (162.7, 85.2)
- moved D15 7.31 mm to (164.8, 84.7)
- moved C2 6.82 mm to (134.2, 49.2)
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Connections:
- C1 pad 1: Net-(U8A-CODEC_VCM) -> /MCU/CODEC_VCM
- J1 pad 2: /MCU/CODEC_LINEOUT -> /MCU/CODEC_VCM
- J1 pad 8: GND -> /MCU/CODEC_LINEOUT
- U8 pad 30: Net-(U8A-CODEC_VCM) -> /MCU/CODEC_VCM
Routing:
- net /MCU/GPIO4_C1_Z: track 0.00 -> 36.8 mm
- net /MCU/CODEC_VCM: track 0.00 -> 33.6 mm, vias 0 -> 2
- net /MCU/FSPI_CS0N: track 20.0 -> 50.2 mm, vias 0 -> 3
- net /MCU/GPIO4_A1_U: track 0.00 -> 29.4 mm, vias 0 -> 2
- net /MCU/GPIO4_A0_U: track 0.00 -> 29.1 mm, vias 0 -> 2
- net /MCU/CODEC_MICBIAS: track 0.00 -> 29.0 mm
- net /MCU/CODEC_MIC0P: track 0.00 -> 26.2 mm
- net /MCU/CODEC_MIC0N: track 0.00 -> 26.2 mm
- net /MCU/GPIO4_A5_U: track 0.00 -> 26.1 mm, vias 0 -> 1
- net /MCU/GPIO2_A5_D: track 0.00 -> 26.1 mm
- net /MCU/GPIO4_A7_U: track 0.00 -> 25.4 mm, vias 0 -> 1
- net /MCU/CODEC_LINEOUT: track 0.00 -> 25.2 mm, vias 0 -> 2
- net /MCU/CODEC_MIC1N: track 0.00 -> 21.8 mm
- net /MCU/CODEC_MIC1P: track 0.00 -> 21.8 mm
- net VBUS: track 2.15 -> 19.8 mm
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- added copper zone on B.Cu, net +BATT

Commit message: feat(Hw):Update_Route
Parts:
- C23, C24, C25, C26, C27, C3, C30, C34, C35, C36, C38, C39, C4, C40, C41, C48, C49, R17, R18, R27, R28, R29, R33, Y2: moved to B.Cu
- J14: value +1V8 -> Conn_01x24; footprint Connector_PinHeader_2.54mm:PinHeader_1x23_P2.54mm_Vertical -> Connector_PinSocket_2.54mm:PinSocket_1x24_P2.54mm_Vertical
- J8: value 3V3 -> Conn_01x24; footprint Connector_PinSocket_2.54mm:PinSocket_1x23_P2.54mm_Vertical -> Connector_PinSocket_2.54mm:PinSocket_1x24_P2.54mm_Vertical
- moved C19 10.4 mm to (155.0, 105.0), turned to 180 degrees
- moved R34 9.86 mm to (138.3, 78.4)
- moved C5 7.08 mm to (128.5, 86.8)
- moved R25 7.08 mm to (128.5, 87.7)
- moved R26 7.08 mm to (128.5, 85.8)
- moved SW3 7.08 mm to (123.7, 86.8)
- moved C60 5.07 mm to (161.2, 83.5), turned to 0 degrees
- moved R9 4.83 mm to (161.2, 82.3), turned to 180 degrees
- moved C34 4.33 mm to (137.7, 107.8), turned to 0 degrees
- moved D1 3.98 mm to (121.2, 91.5), turned to 90 degrees
- moved SW2 3.75 mm to (158.2, 86.8)
- moved R3 3.60 mm to (122.4, 91.5), turned to -90 degrees
- moved C54 2.40 mm to (121.9, 102.7), turned to 180 degrees
- moved C49 2.14 mm to (136.5, 90.4), turned to 90 degrees
- moved R13 1.97 mm to (121.9, 104.5), turned to 180 degrees
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Connections:
- J1 pad 1: +1V8 -> GND
- J1 pad 9: GND -> +1V8
- J14 pad 1: +1V8 -> GND
- J14 pad 10: /MCU/GPIO3_C4_D -> /MCU/GPIO3_B3_D
- J14 pad 11: /MCU/GPIO3_B0_D -> /MCU/GPIO3_B1_D
- J14 pad 12: /MCU/GPIO3_B1_D -> +1V8
- J14 pad 13: /MCU/GPIO3_B2_D -> /MCU/GPIO2_A4_D
- J14 pad 14: /MCU/GPIO3_B3_D -> /MCU/GPIO2_A_2_D
- J14 pad 15: /MCU/GPIO3_B4_D -> /MCU/GPIO2_A0_D_2
- J14 pad 16: /MCU/GPIO3_B5_D -> /MCU/GPIO2_A6_D
- J14 pad 17: /MCU/GPIO3_B6_D -> /MCU/GPIO2_B1_D_2
- J14 pad 18: /MCU/GPIO3_B7_D -> /MCU/GPIO1_C0_D
- J14 pad 19: /MCU/GPIO3_C0_D -> /MCU/GPIO1_C3_D
- J14 pad 2: /MCU/GPIO4_C1_Z -> /MCU/GPIO3_D3_D
- J14 pad 20: /MCU/GPIO3_C1_D -> /MCU/GPIO1_C5_D
- J14 pad 21: /MCU/GPIO3_C2_D -> /MCU/GPIO1_D1_D
- J14 pad 22: /MCU/GPIO3_C3_D -> /MCU/GPIO1_D3_D
- J14 pad 23: GND -> /MCU/GPIO1_C6_D
- J14 pad 3: /MCU/GPIO3_D3_D -> /MCU/GPIO3_D0_D
- J14 pad 4: /MCU/GPIO3_D2_D -> /MCU/GPIO3_C7_D
- J14 pad 5: /MCU/GPIO3_D0_D -> /MCU/GPIO3_C5_D
- J14 pad 6: /MCU/GPIO3_D1_D -> /MCU/GPIO3_C3_D
- J14 pad 7: /MCU/GPIO3_C7_D -> /MCU/GPIO3_C1_D
- J14 pad 8: /MCU/LED -> /MCU/GPIO3_B7_D
- J14 pad 9: /MCU/GPIO3_C5_D -> /MCU/GPIO3_B5_D
- J5 pad 1: +3V3 -> GND
- J5 pad 24: GND -> +3V3
- J8 pad 10: /MCU/GPIO1_C3_D -> /MCU/GPIO2_A3_D
- J8 pad 11: /MCU/GPIO1_C1_D -> /MCU/GPIO2_A5_D
- J8 pad 12: /MCU/GPIO1_C0_D -> +1V8
- J8 pad 13: /MCU/GPIO2_B1_D_1 -> /MCU/GPIO3_B0_D
- J8 pad 14: /MCU/GPIO2_B1_D_2 -> /MCU/GPIO3_B2_D
- J8 pad 15: /MCU/GPIO2_A7_D -> /MCU/GPIO3_B4_D
- J8 pad 16: /MCU/GPIO2_A6_D -> /MCU/GPIO3_B6_D
- J8 pad 17: /MCU/GPIO2_A0_D_1 -> /MCU/GPIO3_C0_D
- J8 pad 18: /MCU/GPIO2_A0_D_2 -> /MCU/GPIO3_C2_D
- J8 pad 19: /MCU/GPIO2_A_2_D -> /MCU/GPIO3_C4_D
- J8 pad 2: /MCU/GPIO1_C6_D -> /MCU/GPIO1_C7_D
- J8 pad 20: /MCU/GPIO2_A3_D -> /MCU/LED
- J8 pad 21: /MCU/GPIO2_A4_D -> /MCU/GPIO3_D1_D
- J8 pad 22: /MCU/GPIO2_A5_D -> /MCU/GPIO3_D2_D
- J8 pad 23: GND -> /MCU/GPIO4_C1_Z
- J8 pad 3: /MCU/GPIO1_C7_D -> /MCU/GPIO1_D2_D
- J8 pad 4: /MCU/GPIO1_D3_D -> /MCU/GPIO1_D0_D
- J8 pad 5: /MCU/GPIO1_D2_D -> /MCU/GPIO1_C4_D
- J8 pad 6: /MCU/GPIO1_D1_D -> /MCU/GPIO1_C1_D
- J8 pad 7: /MCU/GPIO1_D0_D -> /MCU/GPIO2_B1_D_1
- J8 pad 8: /MCU/GPIO1_C5_D -> /MCU/GPIO2_A7_D
- J8 pad 9: /MCU/GPIO1_C4_D -> /MCU/GPIO2_A0_D_1
Routing:
- net VBUS: track 19.8 -> 382.6 mm, vias 0 -> 12
- net +3V3: track 2.97 -> 353.8 mm, vias 0 -> 11
- net +1V8: track 2.49 -> 282.0 mm, vias 0 -> 16
- net /Add-On/SCL: track 0.00 -> 147.3 mm, vias 0 -> 2
- net /Add-On/SDA: track 0.00 -> 145.4 mm, vias 0 -> 2
- net VCC: track 17.2 -> 146.8 mm, vias 0 -> 8
- net /Buck_Converter/v_0.9v: track 5.38 -> 86.6 mm, vias 0 -> 5
- net /Buck_Converter/VCC_DDR: track 4.26 -> 69.1 mm, vias 0 -> 4
- net /MCU/GPIO1_C7_D: track 0.00 -> 61.1 mm
- net /MCU/GPIO1_C6_D: track 0.00 -> 58.6 mm
- net /MCU/GPIO1_D2_D: track 0.00 -> 57.9 mm
- net /MCU/DIN_IR: track 0.00 -> 57.0 mm, vias 0 -> 2
- net /MCU/GPIO1_D3_D: track 0.00 -> 56.1 mm
- net /MCU/GPIO1_D0_D: track 0.00 -> 54.7 mm
- net /MCU/GPIO1_D1_D: track 0.00 -> 52.8 mm
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- added copper zone on B.Cu, net GND
- added copper zone on F.Cu, net GND

Commit message: feat(Hw):Update_Route
Parts:
- moved C39 2.80 mm to (136.1, 90.8)
- moved C48 1.50 mm to (137.0, 90.8)
- moved C49 1.50 mm to (137.9, 90.8)
- moved R28 1.50 mm to (138.9, 90.8)
- moved R2 0.38 mm to (137.7, 106.4)
- moved C29 0.38 mm to (138.6, 106.4)
- moved C25 0.33 mm to (139.8, 90.8)
- moved R36 0.32 mm to (148.5, 111.6)
- moved D2 0.24 mm to (113.1, 96.3)
- moved F1 0.24 mm to (110.2, 96.0)
- moved R27 0.14 mm to (128.4, 98.8)
Routing:
- net +3V3: track 353.8 -> 414.3 mm, vias 11 -> 12
- net GND: track 54.5 -> 92.5 mm, vias 70 -> 102
- net +BATT: track 0.00 -> 15.7 mm
- net /MCU/FSPI_D2: track 40.3 -> 35.0 mm
- net /USB/2_DN: track 11.2 -> 15.3 mm
- net /USB/2_DP: track 11.8 -> 15.3 mm
- net VCC: track 146.8 -> 149.9 mm, vias 8 -> 9
- net /Buck_Converter/v_0.9v: track 86.6 -> 84.8 mm
- net Net-(D4-A): track 0.00 -> 1.48 mm
- net +1V8: track 282.0 -> 280.6 mm
- net /MCU/GPIO3_C4_D: track 38.1 -> 39.5 mm
- net /Buck_Converter/VCC_DDR: track 69.1 -> 70.4 mm
- net /Add-On/SDA: track 145.4 -> 146.4 mm
- net /MCU/GPIO4_A1_U: track 29.5 -> 28.7 mm
- net /Add-On/SCL: track 147.3 -> 148.0 mm
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
Commit message: feat(hw):Updated_review
Parts:
- moved C34 0.63 mm to (137.6, 108.4)
- moved C35 0.45 mm to (137.6, 107.3)
- moved C29 0.38 mm to (139.0, 106.4)
- moved R2 0.36 mm to (138.0, 106.4)
- moved C36 0.26 mm to (137.6, 106.2)
Routing:
- net +3V3: track 414.3 -> 424.3 mm
- net GND: track 92.5 -> 89.2 mm, vias 102 -> 100
- net /Buck_Converter/VCC_DDR: track 70.4 -> 73.4 mm
- net /MCU/DIN_IR: track 57.2 -> 55.0 mm
- net +1V8: track 280.6 -> 282.6 mm
- net /MCU/DEBUG_TX: track 45.4 -> 46.9 mm
- net /Buck_Converter/v_0.9v: track 84.8 -> 85.8 mm
- net /MCU/GPIO3_A6_U: track 48.6 -> 49.6 mm
- net VCC: track 149.9 -> 150.7 mm
- net VBUS: track 382.8 -> 382.1 mm
- net /MCU/GPIO3_A5_U: track 46.6 -> 47.2 mm
- net /MCU/GPIO3_A4_D: track 45.9 -> 45.3 mm
- net /MCU/GPIO3_A7_U: track 49.0 -> 49.6 mm
- net /MCU/GPIO4_A0_U: track 28.7 -> 29.2 mm
