File: hardware/Badge_Bugcon_2025/USB.kicad_sch (KiCad schematic)
At the start: 46 parts, among them J10 Battery, J4 USB_A, J6 USB_A, P4 USB_C_Plug_USB2.0, Q1 DMG3415U-7, SW1 ON, SW4 On, U1 USB3740B-AI9, U2 TP4056, U3 SL2.1A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

Commit message: feat(Hw):Update_Schematic_And_Route
Parts:
- C21, C22: footprint (none) -> Capacitor_SMD:C_0402_1005Metric; LCSC# (none) -> C415703
- C31, C32: footprint (none) -> Capacitor_SMD:C_0402_1005Metric; LCSC# (none) -> C368809
- D12: value MBR120 -> SS34; footprint Diode_SMD:D_SOD-123F -> Diode_SMD:D_SMA; LCSC# C130880 -> C908680; manf# MBR120LSF -> (none)
- D14, D15: value 1N5817 -> SS34; footprint Diode_SMD:D_SOD-123F -> Diode_SMD:D_SMA; LCSC# C727113 -> C908680; manf# 1N5817W -> (none)
- D9: footprint (none) -> Diode_SMD:D_SMA
- F1, F3, F4: value 750mA -> 2A; LCSC# C182438 -> C41380229; manf# 06D0750D -> (none)
- L1: footprint (none) -> Footprints:LQH5BPN
- R44: value 10.6K -> 10.7K; footprint (none) -> Resistor_SMD:R_0402_1005Metric; LCSC# (none) -> C2998172
- R45: footprint (none) -> Resistor_SMD:R_0402_1005Metric; LCSC# (none) -> C2759535
- U4: LCSC# (none) -> C2932326
- U5: value AP2112K-3.3 -> AP2114H-3.3; footprint Package_TO_SOT_SMD:SOT-23-5 -> Package_TO_SOT_SMD:SOT-223-3_TabPin2; LCSC# (none) -> C150716
Connections:
- net +3.3V: now also U5.2 (VOUT); no longer U5.5 (VOUT)
- net +5V: no longer U5.1 (VIN)
- net GND: now also U5.1 (GND); no longer U5.2 (GND)
Changed lines of the file:
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@@
 	)
 	(junction
-		(at 245.11 121.92)
-		(diameter 0)
-		(color 0 0 0 0)
-	)
-	(junction
 		(at 205.74 118.11)
 		(diameter 0)
@@
 	(wire
 		(pts
-			(xy 245.11 124.46) (xy 245.11 121.92)
-		)
-		(stroke
-			(width 0)
-			(type default)
-		)
-	)
-	(wire
-		(pts
 			(xy 90.17 137.16) (xy 91.44 137.16)
 		)
@@
 	(wire
 		(pts
-			(xy 247.65 124.46) (xy 245.11 124.46)
-		)
-		(stroke
-			(width 0)
-			(type default)
-		)
-	)
-	(wire
-		(pts
 			(xy 261.62 54.61) (xy 265.43 54.61)
 		)
@@
 	(wire
 		(pts
-			(xy 245.11 121.92) (xy 241.3 121.92)
+			(xy 241.3 121.92) (xy 247.65 121.92)
 		)
 		(stroke
@@
 	(wire
 		(pts
-			(xy 247.65 121.92) (xy 245.11 121.92)
-		)
-		(stroke
-			(width 0)
-			(type default)
-		)
-	)
-	(wire
-		(pts
 			(xy 265.43 54.61) (xy 265.43 58.42)
 		)
@@
 			)
 		)
-		(property "Footprint" ""
+		(property "Footprint" "Footprints:LQH5BPN"
 			(at 171.45 118.11 0)
 			(effects
@@
 			)
 		)
-		(property "Footprint" ""
+		(property "Footprint" "Resistor_SMD:R_0402_1005Metric"
 			(at 206.502 69.85 90)
 			(effects
@@
 			)
 		)
+		(property "LCSC#" "C2759535"
+			(at 208.28 69.85 0)
+			(effects
+				(font
+					(size 1.27 1.27)
+				)
+				(hide yes)
+			)
+		)
 		(pin "2"
 		)
@@
 			)
 		)
-		(property "Datasheet" "https://www.olimex.com/Products/Breadboarding/BB-PWR-3608/resources/MT3608.pdf"
+		(property "Datasheet" ""
 			(at 165.1 116.84 0)
 			(effects
@@
 			)
 		)
+		(property "LCSC#" "C2932326"
+			(at 171.45 128.27 0)
+			(effects
+				(font
+					(size 1.27 1.27)
+				)
+				(hide yes)
+			)
+		)
 		(pin "3"
 		)
@@
 			)
 		)
-		(property "Value" "10.6K"
+		(property "Value" "10.7K"
 			(at 210.82 58.4199 0)
 			(effects
@@
 			)
 		)
-		(property "Footprint" ""
+		(property "Footprint" "Resistor_SMD:R_0402_1005Metric"
 			(at 206.502 57.15 90)
 			(effects
@@
 			)
 		)
+		(property "LCSC#" "C2998172"
+			(at 208.28 57.15 0)
+			(effects
+				(font
+					(size 1.27 1.27)
+				)
+				(hide yes)
+			)
+		)
 		(pin "2"
 		)
@@
 			)
 		)
-		(property "Value" "1N5817"
+		(property "Value" "SS34"
 			(at 86.36 167.64 0)
 			(effects
@@
 			)
 		)
-		(property "Footprint" "Diode_SMD:D_SOD-123F"
+		(property "Footprint" "Diode_SMD:D_SMA"
 			(at 86.36 165.735 0)
 			(effects
@@
 			)
 		)
-		(property "Datasheet" "http://www.vishay.com/docs/88525/1n5817.pdf"
+		(property "Datasheet" ""
 			(at 86.36 170.18 0)
 			(effects
@@
 			)
 		)
-		(property "manf#" "1N5817W"
+		(property "manf#" ""
 			(at 86.36 170.18 0)
 			(effects
@@
 			)
 		)
-		(property "LCSC#" "C727113"
+		(property "LCSC#" "C908680"
 			(at 86.36 170.18 0)
 			(effects
@@
 			)
 		)
-		(property "Value" "750mA"
+		(property "Value" "2A"
 			(at 46.99 28.0924 0)
 			(effects
@@
 			)
 		)
-		(property "manf#" "06D0750D"
+		(property "manf#" ""
 			(at 46.99 30.48 0)
 			(effects
@@
 			)
 		)
-		(property "LCSC#" "C182438"
+		(property "LCSC#" "C41380229"
 			(at 46.99 30.48 0)
 			(effects
@@
 			)
 		)
-		(property "Value" "MBR120"
+		(property "Value" "SS34"
 			(at 242.443 57.658 0)
 			(effects
@@
 			)
 		)
-		(property "Footprint" "Diode_SMD:D_SOD-123F"
+		(property "Footprint" "Diode_SMD:D_SMA"
 			(at 243.332 50.165 0)
 			(effects
@@
 			)
 		)
-		(property "Datasheet" "http://www.onsemi.com/pub_link/Collateral/MBR340-D.PDF"
+		(property "Datasheet" ""
 			(at 243.332 54.61 0)
 			(effects
@@
 			)
 		)
-		(property "LCSC#" "C130880"
+		(property "LCSC#" "C908680"
 			(at 243.332 54.61 0)
 			(effects
@@
 			)
 		)
-		(property "manf#" "MBR120LSF"
+		(property "manf#" ""
 			(at 243.332 54.61 0)
 			(effects
@@
 			)
 		)
-		(property "Footprint" ""
+		(property "Footprint" "Capacitor_SMD:C_0402_1005Metric"
 			(at 242.2652 130.81 0)
 			(effects
@@
 			)
 		)
+		(property "LCSC#" "C368809"
+			(at 241.3 127 0)
+			(effects
+				(font
+					(size 1.27 1.27)
+				)
+				(hide yes)
+			)
+		)
 		(pin "2"
 		)
@@
 			)
 		)
-		(property "Footprint" ""
+		(property "Footprint" "Capacitor_SMD:C_0402_1005Metric"
 			(at 206.7052 130.81 0)
 			(effects
@@
 			)
 		)
+		(property "LCSC#" "C415703"
+			(at 205.74 127 0)
+			(effects
+				(font
+					(size 1.27 1.27)
+				)
+				(hide yes)
+			)
+		)
 		(pin "2"
 		)
@@
 			)
 		)
-		(property "Value" "750mA"
+		(property "Value" "2A"
 			(at 93.98 134.7724 0)
 			(effects
@@
 			)
 		)
-		(property "manf#" "06D0750D"
+		(property "manf#" ""
 			(at 93.98 137.16 0)
 			(effects
@@
 			)
 		)
-		(property "LCSC#" "C182438"
+		(property "LCSC#" "C41380229"
 			(at 93.98 137.16 0)
 			(effects
@@
 			)
 		)
-		(property "Footprint" ""
+		(property "Footprint" "Capacitor_SMD:C_0402_1005Metric"
 			(at 266.3952 130.81 0)
 			(effects
@@
 			)
 		)
+		(property "LCSC#" "C368809"
+			(at 265.43 127 0)
+			(effects
+				(font
+					(size 1.27 1.27)
+				)
+				(hide yes)
+			)
+		)
 		(pin "1"
 		)
@@
 			)
 		)
-		(property "Footprint" ""
+		(property "Footprint" "Diode_SMD:D_SMA"
 			(at 186.69 118.11 0)
 			(effects
@@
 			)
 		)
-		(property "Datasheet" "~"
+		(property "Datasheet" ""
 			(at 186.69 118.11 0)
 			(effects
@@
 			)
 		)
-		(property "Footprint" ""
+		(property "Footprint" "Capacitor_SMD:C_0402_1005Metric"
 			(at 152.0952 130.81 0)
 			(effects
@@
 			)
 		)
+		(property "LCSC#" "C415703"
+			(at 151.13 127 0)
+			(effects
+				(font
+					(size 1.27 1.27)
+				)
+				(hide yes)
+			)
+		)
 		(pin "1"
 		)
@@
 			)
 		)
-		(property "Value" "AP2112K-3.3"
+		(property "Value" "AP2114H-3.3"
 			(at 255.27 118.11 0)
 			(effects
@@
 			)
 		)
-		(property "Footprint" "Package_TO_SOT_SMD:SOT-23-5"
+		(property "Footprint" "Package_TO_SOT_SMD:SOT-223-3_TabPin2"
 			(at 255.27 116.205 0)
 			(effects
@@
 			)
 		)
-		(property "Datasheet" "https://www.diodes.com/assets/Datasheets/AP2112.pdf"
+		(property "Datasheet" ""
 			(at 255.27 121.92 0)
 			(effects
@@
 			)
 		)
-		(pin "5"
+		(property "LCSC#" "C150716"
+			(at 255.27 124.46 0)
+			(effects
+				(font
+					(size 1.27 1.27)
+				)
+				(hide yes)
+			)
 		)
 		(pin "1"
@@
 			)
 		)
-		(property "Value" "750mA"
+		(property "Value" "2A"
 			(at 93.98 167.7924 0)
 			(effects
@@
 			)
 		)
-		(property "manf#" "06D0750D"
+		(property "manf#" ""
 			(at 93.98 170.18 0)
 			(effects
@@
 			)
 		)
-		(property "LCSC#" "C182438"
+		(property "LCSC#" "C41380229"
 			(at 93.98 170.18 0)
 			(effects
@@
 			)
 		)
-		(property "Value" "1N5817"
+		(property "Value" "SS34"
 			(at 86.36 134.62 0)
 			(effects
@@
 			)
 		)
-		(property "Footprint" "Diode_SMD:D_SOD-123F"
+		(property "Footprint" "Diode_SMD:D_SMA"
 			(at 86.36 132.715 0)
 			(effects
@@
 			)
 		)
-		(property "Datasheet" "http://www.vishay.com/docs/88525/1n5817.pdf"
+		(property "Datasheet" ""
 			(at 86.36 137.16 0)
 			(effects
@@
 			)
 		)
-		(property "manf#" "1N5817W"
+		(property "manf#" ""
 			(at 86.36 137.16 0)
 			(effects
@@
 			)
 		)
-		(property "LCSC#" "C727113"
+		(property "LCSC#" "C908680"
 			(at 86.36 137.16 0)
 			(effects

Commit message: feat(Hw):Update_Route_And_Schematic
Parts:
- removed Y5: 12MHz, Crystal:Crystal_SMD_3225-4Pin_3.2x2.5mm, symbol Device:Crystal
- added Y5: Crystal_GND2, Crystal:Crystal_SMD_3225-4Pin_3.2x2.5mm, symbol Device:Crystal_GND2
Connections:
- net GND: now also Y5.2, Y5.4
- net XIN: now also Y5.3
- net XOUT: now also Y5.1
- net SW: now reaches D9.2 (A), L1.2, U4.1 (SW)
Changed lines of the file:
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@@
 	(wire
 		(pts
+			(xy 50.8 189.23) (xy 50.8 187.96)
+		)
+		(stroke
+			(width 0)
+			(type default)
+		)
+	)
+	(wire
+		(pts
 			(xy 208.28 50.8) (xy 208.28 53.34)
 		)
@@
 		)
 	)
+	(label "SW"
+		(at 179.07 118.11 0)
+		(effects
+			(font
+				(size 1.27 1.27)
+			)
+			(justify left bottom)
+		)
+	)
 	(label "4_DP"
 		(at 63.5 157.48 0)
@@
 	(symbol
 		(lib_id "power:GND")
+		(at 50.8 189.23 0)
+		(unit 1)
+		(exclude_from_sim no)
+		(in_bom yes)
+		(on_board yes)
+		(dnp no)
+		(property "Reference" "#PWR05"
+			(at 50.8 195.58 0)
+			(effects
+				(font
+					(size 1.27 1.27)
+				)
+				(hide yes)
+			)
+		)
+		(property "Value" "GND"
+			(at 50.927 193.6242 0)
+			(effects
+				(font
+					(size 1.27 1.27)
+				)
+			)
+		)
+		(property "Footprint" ""
+			(at 50.8 189.23 0)
+			(effects
+				(font
+					(size 1.27 1.27)
+				)
+				(hide yes)
+			)
+		)
+		(property "Datasheet" ""
+			(at 50.8 189.23 0)
+			(effects
+				(font
+					(size 1.27 1.27)
+				)
+				(hide yes)
+			)
+		)
+		(property "Description" ""
+			(at 50.8 189.23 0)
+			(effects
+				(font
+					(size 1.27 1.27)
+				)
+			)
+		)
+		(pin "1"
+		)
+		(instances
+			(project "Badge_Bugcon_2025"
+				(path "/a95785a0-0aa1-454e-b59f-0ac64970ac71/a5c26cac-72fa-4752-a660-9cd751934916"
+					(reference "#PWR05")
+					(unit 1)
+				)
+			)
+		)
+	)
+	(symbol
+		(lib_id "power:GND")
 		(at 265.43 64.77 0)
 		(unit 1)
@@
 	)
 	(symbol
+		(lib_id "Device:Crystal_GND2")
+		(at 50.8 182.88 0)
+		(mirror y)
+		(unit 1)
+		(exclude_from_sim no)
+		(in_bom yes)
+		(on_board yes)
+		(dnp no)
+		(property "Reference" "Y5"
+			(at 50.8 175.26 0)
+			(effects
+				(font
+					(size 1.27 1.27)
+				)
+			)
+		)
+		(property "Value" "Crystal_GND2"
+			(at 50.8 177.8 0)
+			(effects
+				(font
+					(size 1.27 1.27)
+				)
+			)
+		)
+		(property "Footprint" "Crystal:Crystal_SMD_3225-4Pin_3.2x2.5mm"
+			(at 50.8 182.88 0)
+			(effects
+				(font
+					(size 1.27 1.27)
+				)
+				(hide yes)
+			)
+		)
+		(property "Datasheet" "~"
+			(at 50.8 182.88 0)
+			(effects
+				(font
+					(size 1.27 1.27)
+				)
+				(hide yes)
+			)
+		)
+		(property "Description" "Three pin crystal, GND on pin 2"
+			(at 50.8 182.88 0)
+			(effects
+				(font
+					(size 1.27 1.27)
+				)
+				(hide yes)
+			)
+		)
+		(property "LCSC#" "C133334"
+			(at 50.8 182.88 0)
+			(effects
+				(font
+					(size 1.27 1.27)
+				)
+				(hide yes)
+			)
+		)
+		(pin "2"
+		)
+		(pin "3"
+		)
+		(pin "1"
+		)
+		(pin "4"
+		)
+		(instances
+			(project ""
+				(path "/a95785a0-0aa1-454e-b59f-0ac64970ac71/a5c26cac-72fa-4752-a660-9cd751934916"
+					(reference "Y5")
+					(unit 1)
+				)
+			)
+		)
+	)
+	(symbol
 		(lib_id "power:+5V")
 		(at 205.74 115.57 0)
@@
 					(unit 1)
 				)
-			)
-		)
-	)
-	(symbol
-		(lib_id "Device:Crystal")
-		(at 50.8 182.88 180)
-		(unit 1)
-		(exclude_from_sim no)
-		(in_bom yes)
-		(on_board yes)
-		(dnp no)
-		(property "Reference" "Y5"
-			(at 50.8 186.69 0)
-			(effects
-				(font
-					(size 1.27 1.27)
-				)
-			)
-		)
-		(property "Value" "12MHz"
-			(at 50.8 179.07 0)
-			(effects
-				(font
-					(size 1.27 1.27)
-				)
-			)
-		)
-		(property "Footprint" "Crystal:Crystal_SMD_3225-4Pin_3.2x2.5mm"
-			(at 50.8 182.88 0)
-			(effects
-				(font
-					(size 1.27 1.27)
-				)
-				(hide yes)
-			)
-		)
-		(property "Datasheet" "~"
-			(at 50.8 182.88 0)
-			(effects
-				(font
-					(size 1.27 1.27)
-				)
-				(hide yes)
-			)
-		)
-		(property "Description" "Two pin crystal"
-			(at 50.8 182.88 0)
-			(effects
-				(font
-					(size 1.27 1.27)
-				)
-				(hide yes)
-			)
-		)
-		(property "LCSC#" "C133334"
-			(at 50.8 182.88 0)
-			(effects
-				(font
-					(size 1.27 1.27)
-				)
-				(hide yes)
-			)
-		)
-		(property "Height" ""
-			(at 50.8 182.88 0)
-			(effects
-				(font
-					(size 1.27 1.27)
-				)
-				(hide yes)
-			)
-		)
-		(property "Manufacturer_Name" ""
-			(at 50.8 182.88 0)
-			(effects
-				(font
-					(size 1.27 1.27)
-				)
-				(hide yes)
-			)
-		)
-		(property "Mouser Part Number" ""
-			(at 50.8 182.88 0)
-			(effects
-				(font
-					(size 1.27 1.27)
-				)
-				(hide yes)
-			)
-		)
-		(property "Mouser Price/Stock" ""
-			(at 50.8 182.88 0)
-			(effects
-				(font
-					(size 1.27 1.27)
-				)
-				(hide yes)
-			)
-		)
-		(property "Availability" ""
-			(at 50.8 182.88 0)
-			(effects
-				(font
-					(size 1.27 1.27)
-				)
-				(hide yes)
-			)
-		)
-		(property "Check_prices" ""
-			(at 50.8 182.88 0)
-			(effects
-				(font
-					(size 1.27 1.27)
-				)
-				(hide yes)
-			)
-		)
-		(property "Description_1" ""
-			(at 50.8 182.88 0)
-			(effects
-				(font
-					(size 1.27 1.27)
-				)
-				(hide yes)
-			)
-		)
-		(property "MANUFACTURER" ""
-			(at 50.8 182.88 0)
-			(effects
-				(font
-					(size 1.27 1.27)
-				)
-				(hide yes)
-			)
-		)
-		(property "MAXIMUM_PACKAGE_HEIGHT" ""
-			(at 50.8 182.88 0)
-			(effects
-				(font
-					(size 1.27 1.27)
-				)
-				(hide yes)
-			)
-		)
-		(property "MF" ""
-			(at 50.8 182.88 0)
-			(effects
-				(font
-					(size 1.27 1.27)
-				)
-				(hide yes)
-			)
-		)
-		(property "MP" ""
-			(at 50.8 182.88 0)
-			(effects
-				(font
-					(size 1.27 1.27)
-				)
-				(hide yes)
-			)
-		)
-		(property "PARTREV" ""
-			(at 50.8 182.88 0)
-			(effects
-				(font
-					(size 1.27 1.27)
-				)
-				(hide yes)
-			)
-		)
-		(property "Package" ""
-			(at 50.8 182.88 0)
-			(effects
-				(font
-					(size 1.27 1.27)
-				)
-				(hide yes)
-			)
-		)
-		(property "Price" ""
-			(at 50.8 182.88 0)
-			(effects
-				(font
-					(size 1.27 1.27)
-				)
-				(hide yes)
-			)
-		)
-		(property "STANDARD" ""
-			(at 50.8 182.88 0)
-			(effects
-				(font
-					(size 1.27 1.27)
-				)
-				(hide yes)
-			)
-		)
-		(property "SnapEDA_Link" ""
-			(at 50.8 182.88 0)
-			(effects
-				(font
-					(size 1.27 1.27)
-				)
-				(hide yes)
-			)
-		)
-		(property "JLCPCB" ""
-			(at 50.8 182.88 0)
-			(effects
-				(font
-					(size 1.27 1.27)
-				)
-				(hide yes)
-			)
-		)
-		(property "Manufacter Number" ""
-			(at 50.8 182.88 0)
-			(effects
-				(font
-					(size 1.27 1.27)
-				)
-				(hide yes)
-			)
-		)
-		(pin "1"
-		)
-		(pin "3"
-		)
-		(instances
-			(project "Badge_Bugcon_2025"
-				(path "/a95785a0-0aa1-454e-b59f-0ac64970ac71/a5c26cac-72fa-4752-a660-9cd751934916"
-					(reference "Y5")
-					(unit 1)
-				)

Commit message: feat(Hw):Update_USB_Selector
Parts:
- removed U1: USB3740B-AI9, Package_DFN_QFN:UQFN-10_1.3x1.8mm_P0.4mm, symbol Interface_USB:USB3740B-AI9
- added U1: FSUSB30MUX, Footprints:IC_FSUSB42UMX, symbol Interface_USB:FSUSB30MUX
- SW1: manf# SK12D07VG4 -> (none)
- SW4: footprint Footprints:MSK12C02 -> Button_Switch_THT:SW_Slide_SPDT_Angled_CK_OS102011MA1Q; LCSC# C431540 -> C393937
Connections:
- net +5V: now also U1.9 (VCC)
- net 1_DN: now also U1.6 (HSD2-)
- net 1_DP: now also U1.7 (HSD2+)
- net 2_DN: now also U1.4 (HSD1-)
- net 2_DP: now also U1.5 (HSD1+)
- net D+: now also U1.1 (D+)
- net D-: now also U1.2 (D-)
- net GND: now also U1.3 (GND), U1.8 (~{OE})
- net S: now also U1.10 (S)

Commit message: feat(Hw):Update_Route
Parts:
- SW4: value On -> USB Selector
Changed lines of the file:
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@@
 			)
 		)
-		(property "Value" "On"
+		(property "Value" "USB Selector"
 			(at 72.39 100.4824 0)
 			(effects

Commit message: update connections same image layer
Parts:
- added R46: 10K, Resistor_SMD:R_0402_1005Metric, symbol Device:R
Connections:
- net +5V: no longer C31.1, U5.3 (VIN)
- net Enable: now also R46.2
- net VCC: now also C31.1, U5.3 (VIN)
- new net +3V3: R46.1
Changed lines of the file:
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@@
 	)
 	(junction
+		(at 147.32 60.96)
+		(diameter 0)
+		(color 0 0 0 0)
+	)
+	(junction
 		(at 241.3 121.92)
 		(diameter 0)
@@
 	(wire
 		(pts
+			(xy 147.32 59.69) (xy 147.32 60.96)
+		)
+		(stroke
+			(width 0)
+			(type default)
+		)
+	)
+	(wire
+		(pts
 			(xy 236.347 54.61) (xy 236.347 58.801)
 		)
@@
 	(wire
 		(pts
+			(xy 147.32 60.96) (xy 144.78 60.96)
+		)
+		(stroke
+			(width 0)
+			(type default)
+		)
+	)
+	(wire
+		(pts
 			(xy 191.77 130.81) (xy 191.77 133.35)
 		)
@@
 	(wire
 		(pts
+			(xy 147.32 49.53) (xy 147.32 52.07)
+		)
+		(stroke
+			(width 0)
+			(type default)
+		)
+	)
+	(wire
+		(pts
 			(xy 81.28 135.89) (xy 81.28 137.16)
 		)
@@
 	(wire
 		(pts
-			(xy 157.48 60.96) (xy 156.21 60.96)
+			(xy 157.48 60.96) (xy 147.32 60.96)
 		)
 		(stroke
@@
 	(hierarchical_label "Enable"
 		(shape input)
-		(at 156.21 60.96 180)
+		(at 144.78 60.96 180)
 		(effects
 			(font
@@
 		(on_board yes)
 		(dnp no)
-		(fields_autoplaced yes)
 		(property "Reference" "D16"
-			(at 146.05 59.69 0)
+			(at 140.97 64.77 0)
 			(effects
 				(font
@@
 		)
 		(property "Value" "LED"
-			(at 146.05 62.23 0)
+			(at 140.97 67.31 0)
 			(effects
 				(font
@@
 	)
 	(symbol
-		(lib_id "power:+5V")
-		(at 241.3 119.38 0)
-		(unit 1)
-		(exclude_from_sim no)
-		(in_bom yes)
-		(on_board yes)
-		(dnp no)
-		(fields_autoplaced yes)
-		(property "Reference" "#PWR039"
-			(at 241.3 123.19 0)
-			(effects
-				(font
-					(size 1.27 1.27)
-				)
-				(hide yes)
-			)
-		)
-		(property "Value" "+5V"
-			(at 241.3 114.3 0)
-			(effects
-				(font
-					(size 1.27 1.27)
-				)
-			)
-		)
-		(property "Footprint" ""
-			(at 241.3 119.38 0)
-			(effects
-				(font
-					(size 1.27 1.27)
-				)
-				(hide yes)
-			)
-		)
-		(property "Datasheet" ""
-			(at 241.3 119.38 0)
-			(effects
-				(font
-					(size 1.27 1.27)
-				)
-				(hide yes)
-			)
-		)
-		(property "Description" "Power symbol creates a global label with name \"+5V\""
-			(at 241.3 119.38 0)
-			(effects
-				(font
-					(size 1.27 1.27)
-				)
-				(hide yes)
-			)
-		)
-		(pin "1"
-		)
-		(instances
-			(project "Badge_Bugcon_2025"
-				(path "/a95785a0-0aa1-454e-b59f-0ac64970ac71/a5c26cac-72fa-4752-a660-9cd751934916"
-					(reference "#PWR039")
-					(unit 1)
-				)
-			)
-		)
-	)
-	(symbol
 		(lib_id "power:GND")
 		(at 205.74 133.35 0)
@@
 	)
 	(symbol
+		(lib_id "power:+3V3")
+		(at 147.32 49.53 0)
+		(unit 1)
+		(exclude_from_sim no)
+		(in_bom yes)
+		(on_board yes)
+		(dnp no)
+		(fields_autoplaced yes)
+		(property "Reference" "#PWR0115"
+			(at 147.32 53.34 0)
+			(effects
+				(font
+					(size 1.27 1.27)
+				)
+				(hide yes)
+			)
+		)
+		(property "Value" "+3V3"
+			(at 147.32 44.45 0)
+			(effects
+				(font
+					(size 1.27 1.27)
+				)
+			)
+		)
+		(property "Footprint" ""
+			(at 147.32 49.53 0)
+			(effects
+				(font
+					(size 1.27 1.27)
+				)
+				(hide yes)
+			)
+		)
+		(property "Datasheet" ""
+			(at 147.32 49.53 0)
+			(effects
+				(font
+					(size 1.27 1.27)
+				)
+				(hide yes)
+			)
+		)
+		(property "Description" "Power symbol creates a global label with name \"+3V3\""
+			(at 147.32 49.53 0)
+			(effects
+				(font
+					(size 1.27 1.27)
+				)
+				(hide yes)
+			)
+		)
+		(pin "1"
+		)
+		(instances
+			(project "Badge_Bugcon_2025"
+				(path "/a95785a0-0aa1-454e-b59f-0ac64970ac71/a5c26cac-72fa-4752-a660-9cd751934916"
+					(reference "#PWR0115")
+					(unit 1)
+				)
+			)
+		)
+	)
+	(symbol
 		(lib_id "Regulator_Switching:MT3608")
 		(at 171.45 128.27 0)
@@
 	)
 	(symbol
+		(lib_id "power:VCC")
+		(at 241.3 119.38 0)
+		(unit 1)
+		(exclude_from_sim no)
+		(in_bom yes)
+		(on_board yes)
+		(dnp no)
+		(fields_autoplaced yes)
+		(property "Reference" "#PWR0101"
+			(at 241.3 123.19 0)
+			(effects
+				(font
+					(size 1.27 1.27)
+				)
+				(hide yes)
+			)
+		)
+		(property "Value" "VCC"
+			(at 241.3 114.3 0)
+			(effects
+				(font
+					(size 1.27 1.27)
+				)
+			)
+		)
+		(property "Footprint" ""
+			(at 241.3 119.38 0)
+			(effects
+				(font
+					(size 1.27 1.27)
+				)
+				(hide yes)
+			)
+		)
+		(property "Datasheet" ""
+			(at 241.3 119.38 0)
+			(effects
+				(font
+					(size 1.27 1.27)
+				)
+				(hide yes)
+			)
+		)
+		(property "Description" "Power symbol creates a global label with name \"VCC\""
+			(at 241.3 119.38 0)
+			(effects
+				(font
+					(size 1.27 1.27)
+				)
+				(hide yes)
+			)
+		)
+		(pin "1"
+		)
+		(instances
+			(project "Badge_Bugcon_2025"
+				(path "/a95785a0-0aa1-454e-b59f-0ac64970ac71/a5c26cac-72fa-4752-a660-9cd751934916"
+					(reference "#PWR0101")
+					(unit 1)
+				)
+			)
+		)
+	)
+	(symbol
 		(lib_id "Device:R")
 		(at 208.28 57.15 0)
@@
 					(unit 1)
 				)
+			)
+		)
+	)
+	(symbol
+		(lib_id "Device:R")
+		(at 147.32 55.88 0)
+		(unit 1)
+		(exclude_from_sim no)
+		(in_bom yes)
+		(on_board yes)
+		(dnp no)
+		(fields_autoplaced yes)
+		(property "Reference" "R46"
+			(at 149.86 54.6099 0)
+			(effects
+				(font
+					(size 1.27 1.27)
+				)
+				(justify left)
+			)
+		)
+		(property "Value" "10K"
+			(at 149.86 57.1499 0)
+			(effects
+				(font
+					(size 1.27 1.27)
+				)
+				(justify left)
+			)
+		)
+		(property "Footprint" "Resistor_SMD:R_0402_1005Metric"
+			(at 145.542 55.88 90)
+			(effects
+				(font
+					(size 1.27 1.27)
+				)
+				(hide yes)
+			)
+		)
+		(property "Datasheet" "~"
+			(at 147.32 55.88 0)
+			(effects
+				(font
+					(size 1.27 1.27)
+				)
+				(hide yes)
+			)
+		)
+		(property "Description" "Resistor"
+			(at 147.32 55.88 0)
+			(effects
+				(font
+					(size 1.27 1.27)
+				)
+				(hide yes)
+			)
+		)
+		(property "JLCPCB" ""
+			(at 147.32 55.88 0)
+			(effects
+				(font
+					(size 1.27 1.27)
+				)
+				(hide yes)
+			)
+		)
+		(property "Manufacter Number" ""
+			(at 147.32 55.88 0)
+			(effects
+				(font
+					(size 1.27 1.27)
+				)
+				(hide yes)
+			)
+		)
+		(property "LCSC#" "C2759535"
+			(at 147.32 55.88 0)
+			(effects
+				(font
+					(size 1.27 1.27)
+				)
+				(hide yes)
+			)
+		)
+		(pin "2"
+		)
+		(pin "1"
+		)
+		(instances
+			(project "Badge_Bugcon_2025"
+				(path "/a95785a0-0aa1-454e-b59f-0ac64970ac71/a5c26cac-72fa-4752-a660-9cd751934916"
+					(reference "R46")
+					(unit 1)
+				)
